File: boards/MC3_COL_MAIN_V1.0/MotorChannel.kicad_sch (KiCad schematic)
At the start: 7 parts, among them J1 MOTOR, U1 DRV8214RTER

Commit message: Schematic annotated in eeschema (per-instance references for the 4 channel sheets); user review OK
Co-Authored-By: Claude Fable 5 <noreply@anthropic.com>
Parts:
- renumbered C1 to C14, C2 to C15, J1 to J7, R1 to R10, R2 to R11, R3 to R12, U1 to U3

Commit message: Schematic re-annotated in eeschema after yaw channel + strap pull-ups
Co-Authored-By: Claude Fable 5 <noreply@anthropic.com>
Parts:
- renumbered R10 to R14, R11 to R15, R12 to R16
Changed lines of the file:
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@@
 		(in_pos_files yes)
 		(dnp no)
-		(property "Reference" "R11"
+		(property "Reference" "R15"
 			(at 136.652 64.77 90)
 			(show_name no)
@@
 			(project "MC3_COL_MAIN_V1.0"
 				(path "/7d5f4202-d55e-4c7b-a2df-dd599db38e48/5db6fbb9-0012-419b-b34a-9d86ac1f5217"
-					(reference "R14")
+					(reference "R18")
 					(unit 1)
 				)
 				(path "/7d5f4202-d55e-4c7b-a2df-dd599db38e48/8cfd3b4a-99dc-4b05-a7ad-f8199ec40931"
-					(reference "R23")
+					(reference "R27")
 					(unit 1)
 				)
 				(path "/7d5f4202-d55e-4c7b-a2df-dd599db38e48/9d20a086-3ce1-4783-a1c3-78685ff35655"
-					(reference "R20")
+					(reference "R24")
 					(unit 1)
 				)
 				(path "/7d5f4202-d55e-4c7b-a2df-dd599db38e48/a93ffbcb-09b2-46f4-87ff-b0a1b53638e4"
-					(reference "R11")
+					(reference "R15")
 					(unit 1)
 				)
 				(path "/7d5f4202-d55e-4c7b-a2df-dd599db38e48/f0c3363d-cc6b-4f74-be1d-ed0c2c093cdf"
-					(reference "R17")
+					(reference "R21")
 					(unit 1)
 				)
@@
 		(in_pos_files yes)
 		(dnp no)
-		(property "Reference" "R12"
+		(property "Reference" "R16"
 			(at 146.812 64.77 90)
 			(show_name no)
@@
 			(project "MC3_COL_MAIN_V1.0"
 				(path "/7d5f4202-d55e-4c7b-a2df-dd599db38e48/5db6fbb9-0012-419b-b34a-9d86ac1f5217"
-					(reference "R15")
+					(reference "R19")
 					(unit 1)
 				)
 				(path "/7d5f4202-d55e-4c7b-a2df-dd599db38e48/8cfd3b4a-99dc-4b05-a7ad-f8199ec40931"
-					(reference "R24")
+					(reference "R28")
 					(unit 1)
 				)
 				(path "/7d5f4202-d55e-4c7b-a2df-dd599db38e48/9d20a086-3ce1-4783-a1c3-78685ff35655"
-					(reference "R21")
+					(reference "R25")
 					(unit 1)
 				)
 				(path "/7d5f4202-d55e-4c7b-a2df-dd599db38e48/a93ffbcb-09b2-46f4-87ff-b0a1b53638e4"
-					(reference "R12")
+					(reference "R16")
 					(unit 1)
 				)
 				(path "/7d5f4202-d55e-4c7b-a2df-dd599db38e48/f0c3363d-cc6b-4f74-be1d-ed0c2c093cdf"
-					(reference "R18")
+					(reference "R22")
 					(unit 1)
 				)
@@
 		(in_pos_files yes)
 		(dnp no)
-		(property "Reference" "R10"
+		(property "Reference" "R14"
 			(at 126.492 91.44 90)
 			(show_name no)
@@
 			(project "MC3_COL_MAIN_V1.0"
 				(path "/7d5f4202-d55e-4c7b-a2df-dd599db38e48/5db6fbb9-0012-419b-b34a-9d86ac1f5217"
-					(reference "R13")
+					(reference "R17")
 					(unit 1)
 				)
 				(path "/7d5f4202-d55e-4c7b-a2df-dd599db38e48/8cfd3b4a-99dc-4b05-a7ad-f8199ec40931"
-					(reference "R22")
+					(reference "R26")
 					(unit 1)
 				)
 				(path "/7d5f4202-d55e-4c7b-a2df-dd599db38e48/9d20a086-3ce1-4783-a1c3-78685ff35655"
-					(reference "R19")
+					(reference "R23")
 					(unit 1)
 				)
 				(path "/7d5f4202-d55e-4c7b-a2df-dd599db38e48/a93ffbcb-09b2-46f4-87ff-b0a1b53638e4"
-					(reference "R10")
+					(reference "R14")
 					(unit 1)
 				)
 				(path "/7d5f4202-d55e-4c7b-a2df-dd599db38e48/f0c3363d-cc6b-4f74-be1d-ed0c2c093cdf"
-					(reference "R16")
-					(unit 1)
-				)
+					(reference "R20")
+					(unit 1)
+				)

Commit message: Design review changes: HSE caps 33pF, R_IPROPI 6.8k (1.99 A trip), VM bulk, sensor rail filter, input fuse+TVS, NRST cap, 6-pin SWD with SWO, VDDA ferrite, LEDs, test points, tantalum LDO cap
- MCU: C6/C10 18pF -> 33pF (X32258MSB4SI is CL=20pF); C60 100nF on NRST; J2 -> Conn_01x06
  (+NRST, +SWO on PB3); VDDA split from +3V3 through FB60 + PWR_FLAG; heartbeat LED D60/R60
  on PA5, power LED D61/R61; test points TP60-64 (+3V3, SCL, SDA, IPROPI_leaf1, GND)
- Power: J1 -> VIN_PAD -> F60 polyfuse -> VIN_PROT; D62 SMAJ5.0A TVS VIN_PROT-GND; C61/C62
  2x22uF VM bulk; TP65 VM, TP66 VIN_PROT; C2 LDO output cap -> tantalum 22uF 10V (C_Polarized,
  CP_EIA-3216-18)
- Connectors: FFC VIN now VSENS = VM through FB61 + C63 4.7uF
- MotorChannel: R_IPROPI 8.45k -> 6.8k (I_TRIP = 3.3/(6.8k*244uA/A) = 1.99 A)
- Library: stock L_0603, D_SMA, Fuse_1206, CP_EIA-3216-18, TestPoint_Pad_1.0x1.0mm, LED_0603,
  PinHeader_1x06 footprints copied in
- ERC 0 errors (same_local_global_label warnings only); netlist walked

Co-Authored-By: Claude Fable 5 <noreply@anthropic.com>
Parts:
- R14: value 8.45k -> 6.8k; Note PROVISIONAL R_IPROPI = 8.45k (SLVSH04 Table 9-1 example). D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 -> R_IPROPI 6.8k: I_TRIP = VREF/(R*A_IPROPI) = 3.3/(6.8k*244uA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
Other:
- note added: "Review 2026-08-22: R_IPROPI 6.8k -> hardware current trip 1.99 A (was 8.45k -> 1.60 A)."
Changed lines of the file:
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@@
 		)
 	)
+  (text "Review 2026-08-22: R_IPROPI 6.8k -> hardware current trip 1.99 A (was 8.45k -> 1.60 A)."
+    (at 40 120 0)
+    (effects (font (size 1.5 1.5)))
+  )
 	(symbol
 		(lib_id "Device:R")
@@
 			)
 		)
-		(property "Value" "8.45k"
+		(property "Value" "6.8k"
 			(at 124.46 91.44 90)
 			(show_name no)
@@
 			)
 		)
-		(property "Note" "PROVISIONAL R_IPROPI = 8.45k (SLVSH04 Table 9-1 example). Derive from CS_GAIN_SEL=000b range and ADC full scale - CALC owed to vault"
-			(at 124.46 91.44 0)
-			(hide yes)
+		(property "Note" "R_IPROPI 6.8k: I_TRIP = VREF/(R*A_IPROPI) = 3.3/(6.8k*244uA/A) = 1.99 A (DRV8214 2 A RMS rating; SLVSH04 eq. 3, A_IPROPI_H = 244 uA/A at CS_GAIN_SEL=000b). V_IPROPI at 1.65 A stall = 2.74 V (ADC headroom). PROVISIONAL -> vault CALC"
+			(at 124.46 91.44 0)
+			(hide yes)

Commit message: LCSC/MPN fields on every support part (verified against the JLCPCB DB); R_IPROPI 6.8k = C93940; polyfuse 1206L200/12NR; MIGRATION register
Co-Authored-By: Claude Fable 5 <noreply@anthropic.com>
Parts:
- C14: LCSC (none) -> C15849; MPN (none) -> CL10A105KB8NNNC
- C15: LCSC (none) -> C1525; MPN (none) -> CL05B104KO5NNNC
- R14: LCSC (none) -> C93940; MPN (none) -> RC0402FR-076K8L
- R15, R16: LCSC (none) -> C25744; MPN (none) -> 0402WGF1002TCE
Changed lines of the file:
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@@
 			)
 		)
-	)
+		(property "LCSC" "C25744"
+			(at 134.62 64.77 0)
+			(hide yes)
+			(effects
+				(font
+					(size 1.27 1.27)
+				)
+			)
+		)
+		(property "MPN" "0402WGF1002TCE"
+			(at 134.62 64.77 0)
+			(hide yes)
+			(effects
+				(font
+					(size 1.27 1.27)
+				)
+			)
+		))
 	(symbol
 		(lib_id "Device:R")
@@
 			)
 		)
-	)
+		(property "LCSC" "C25744"
+			(at 144.78 64.77 0)
+			(hide yes)
+			(effects
+				(font
+					(size 1.27 1.27)
+				)
+			)
+		)
+		(property "MPN" "0402WGF1002TCE"
+			(at 144.78 64.77 0)
+			(hide yes)
+			(effects
+				(font
+					(size 1.27 1.27)
+				)
+			)
+		))
 	(symbol
 		(lib_id "Device:R")
@@
 			)
 		)
-	)
+		(property "LCSC" "C93940"
+			(at 124.46 91.44 0)
+			(hide yes)
+			(effects
+				(font
+					(size 1.27 1.27)
+				)
+			)
+		)
+		(property "MPN" "RC0402FR-076K8L"
+			(at 124.46 91.44 0)
+			(hide yes)
+			(effects
+				(font
+					(size 1.27 1.27)
+				)
+			)
+		))
 	(symbol
 		(lib_id "power:GND")
@@
 			)
 		)
-	)
+		(property "LCSC" "C15849"
+			(at 80.01 58.42 0)
+			(hide yes)
+			(effects
+				(font
+					(size 1.27 1.27)
+				)
+			)
+		)
+		(property "MPN" "CL10A105KB8NNNC"
+			(at 80.01 58.42 0)
+			(hide yes)
+			(effects
+				(font
+					(size 1.27 1.27)
+				)
+			)
+		))
 	(symbol
 		(lib_id "MC3_COL_MAIN:DRV8214RTER")
@@
 			)
 		)
-	)
+		(property "LCSC" "C1525"
+			(at 119.38 58.42 0)
+			(hide yes)
+			(effects
+				(font
+					(size 1.27 1.27)
+				)
+			)
+		)
+		(property "MPN" "CL05B104KO5NNNC"
+			(at 119.38 58.42 0)
+			(hide yes)
+			(effects
+				(font
+					(size 1.27 1.27)
+				)
+			)
+		))
 )

Commit message: MCU -> STM32F412RET6 (pin-identical, adds bxCAN); CAN sheet: TJA1051T/3, split termination + jumper, PESD1CAN, CANH/CANL/GND pads
- MCU: U2 symbol MC3_COL_MAIN:STM32F412RET6 (same pin map as the F411), LCSC C89374; CAN1_RX PA11,
  CAN1_TX PA12; RC_OUT_leaf4 moved PA11 -> PB14
- CAN.kicad_sch (root sheet 'CAN'): U70 TJA1051T/3 (C38695) VCC from VM via FB62 + C70/C71,
  VIO +3V3, S low; JP70 solder jumper (bridged) -> R70/R71 62R split termination with C72 4.7nF;
  D70 PESD1CAN (C15771); J70 3 bare pads CANH/CANL/GND (new footprint SolderPads_3x)
- Library: STM32F412RET6 symbol; SolderPads_3x_2.2x1.4mm_P2.6mm, SOT-23, SolderJumper-2 footprints
- ERC 0 errors; netlist checked

Co-Authored-By: Claude Fable 5 <noreply@anthropic.com>
Parts:
- renumbered C14 to C18, C15 to C19, R14 to R16, R15 to R17, R16 to R18
