File: boards/MC3_COL_MAIN_V1.0/Power.kicad_sch (KiCad schematic)
At the start: 12 parts, among them J1 SUPPLY_IN, Q1 AO4407C, U1 AMS1117-3.3

Commit message: MCU -> STM32F412RET6 (pin-identical, adds bxCAN); CAN sheet: TJA1051T/3, split termination + jumper, PESD1CAN, CANH/CANL/GND pads
- MCU: U2 symbol MC3_COL_MAIN:STM32F412RET6 (same pin map as the F411), LCSC C89374; CAN1_RX PA11,
  CAN1_TX PA12; RC_OUT_leaf4 moved PA11 -> PB14
- CAN.kicad_sch (root sheet 'CAN'): U70 TJA1051T/3 (C38695) VCC from VM via FB62 + C70/C71,
  VIO +3V3, S low; JP70 solder jumper (bridged) -> R70/R71 62R split termination with C72 4.7nF;
  D70 PESD1CAN (C15771); J70 3 bare pads CANH/CANL/GND (new footprint SolderPads_3x)
- Library: STM32F412RET6 symbol; SolderPads_3x_2.2x1.4mm_P2.6mm, SOT-23, SolderJumper-2 footprints
- ERC 0 errors; netlist checked

Co-Authored-By: Claude Fable 5 <noreply@anthropic.com>
Parts:
- renumbered C61 to C3, C62 to C4, D62 to D1, F60 to F1, TP65 to TP1, TP66 to TP2
