File: boards/MC3_COL_MAIN_V1.0/Connectors.kicad_sch (KiCad schematic)
At the start: 8 parts, among them J4 ENC_leaf1, J5 ENC_leaf2, J6 ENC_leaf3, J7 ENC_leaf4

Commit message: Schematic: root sheet on-grid, I2C address straps as GND/+3V3 global labels, ERC clean (warnings only)
- Root: Power/MCU/Connectors + 4x MotorChannel instances on the 1.27 mm grid; sheet pins wired
  to EN/PH/IPROPI/RC_OUT/nFAULT_leafN global labels; A1/A0 straps leaf1 GND/GND, leaf2
  GND/+3V3, leaf3 +3V3/GND, leaf4 +3V3/+3V3 (PROVISIONAL)
- Connectors: removed a GND drop that shorted ENC_leaf4; VM on the FFCs as global labels
- Power: PWR_FLAGs placed on the pin ends (VIN_PROT, VM, GND)
- ERC (kicad-cli, all severities): 0 errors, 8 same_local_global_label warnings (intended)
- Reference designators still duplicated across the 4 channel instances: needs Annotate
  in eeschema (no CLI path)

Co-Authored-By: Claude Fable 5 <noreply@anthropic.com>
Connections:
- net GND: no longer J7.3 (Pin_3), R33.2
- new net ENC_leaf4: J7.3 (Pin_3), R33.2
Changed lines of the file:
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@@
 	(generator_version "10.0")
 	(paper "A4")
-	(junction
-		(at 52.07 172.72)
-		(diameter 0)
-	)
 	(no_connect
 		(at 54.61 54.61)
@@
 	(wire
 		(pts
-			(xy 52.07 170.18)
-			(xy 52.07 180.34)
-		)
-	)
-	(label "VM"
-		(at 54.61 46.99 180)
-		(effects
-			(font
-				(size 1.27 1.27)
-			)
-			(justify right bottom)
-		)
-	)
-	(label "VM"
-		(at 54.61 87.63 180)
-		(effects
-			(font
-				(size 1.27 1.27)
-			)
-			(justify right bottom)
-		)
-	)
-	(label "VM"
-		(at 54.61 127 180)
-		(effects
-			(font
-				(size 1.27 1.27)
-			)
-			(justify right bottom)
-		)
-	)
-	(label "VM"
-		(at 54.61 167.64 180)
-		(effects
-			(font
-				(size 1.27 1.27)
-			)
-			(justify right bottom)
+			(xy 54.61 46.99)
+			(xy 52.07 46.99)
+		)
+	)
+	(wire
+		(pts
+			(xy 54.61 87.63)
+			(xy 52.07 87.63)
+		)
+	)
+	(wire
+		(pts
+			(xy 54.61 127)
+			(xy 52.07 127)
+		)
+	)
+	(wire
+		(pts
+			(xy 54.61 167.64)
+			(xy 52.07 167.64)
+		)
+	)
+	(wire
+		(pts
+			(xy 54.61 49.53)
+			(xy 44.45 49.53)
+		)
+	)
+	(text "Encoder interface - four 0.5 mm FFCs, one per leaf, to the LX34311 sensor boards (COL-COTS-0016). Contract: VIN 4-6 V from VM, GND, SIG open-drain pulled to +3V3 here (10k), spare unassigned. Vault: Main-Board-01 Encoder Interface / Connectors. Motor pads are on the MotorChannel sheet; supply pads on Power."
+		(at 30 25 0)
+		(effects
+			(font
+				(size 1.5 1.5)
+			)
 		)
 	)
@@
 		)
 	)
-  (text "Encoder interface - four 0.5 mm FFCs, one per leaf, to the LX34311 sensor boards (COL-COTS-0016). Contract: VIN 4-6 V from VM, GND, SIG open-drain pulled to +3V3 here (10k), spare unassigned. Vault: Main-Board-01 Encoder Interface / Connectors. Motor pads are on the MotorChannel sheet; supply pads on Power."
-    (at 30 25 0)
-    (effects (font (size 1.5 1.5)))
-  )
+	(global_label "VM"
+		(shape input)
+		(at 52.07 46.99 180)
+		(effects
+			(font
+				(size 1.27 1.27)
+			)
+			(justify right)
+		)
+	)
+	(global_label "VM"
+		(shape input)
+		(at 52.07 87.63 180)
+		(effects
+			(font
+				(size 1.27 1.27)
+			)
+			(justify right)
+		)
+	)
+	(global_label "VM"
+		(shape input)
+		(at 52.07 127 180)
+		(effects
+			(font
+				(size 1.27 1.27)
+			)
+			(justify right)
+		)
+	)
+	(global_label "VM"
+		(shape input)
+		(at 52.07 167.64 180)
+		(effects
+			(font
+				(size 1.27 1.27)
+			)
+			(justify right)
+		)
+	)
 	(symbol
 		(lib_id "Connector_Generic:Conn_01x04")
@@
 			)
 		)
+		(property "LCSC" "C425129"
+			(at 59.69 49.53 0)
+			(hide yes)
+			(effects
+				(font
+					(size 1.27 1.27)
+				)
+			)
+		)
+		(property "MPN" "AYF530435"
+			(at 59.69 49.53 0)
+			(hide yes)
+			(effects
+				(font
+					(size 1.27 1.27)
+				)
+			)
+		)
+		(property "Note" "Encoder FFC leaf1: 1 VIN(VM) 2 GND 3 SIG 4 spare. No COTS record (support part) - vault Connectors / Encoder Interface"
+			(at 59.69 49.53 0)
+			(hide yes)
+			(effects
+				(font
+					(size 1.27 1.27)
+				)
+			)
+		)
 		(instances
 			(project "Connectors"
@@
 			)
 		)
-		(property "LCSC" "C425129"
-			(at 59.69 49.53 0)
-			(hide yes)
-			(effects
-				(font
-					(size 1.27 1.27)
-				)
-			)
-		)
-		(property "MPN" "AYF530435"
-			(at 59.69 49.53 0)
-			(hide yes)
-			(effects
-				(font
-					(size 1.27 1.27)
-				)
-			)
-		)
-		(property "Note" "Encoder FFC leaf1: 1 VIN(VM) 2 GND 3 SIG 4 spare. No COTS record (support part) - vault Connectors / Encoder Interface"
-			(at 59.69 49.53 0)
-			(hide yes)
-			(effects
-				(font
-					(size 1.27 1.27)
-				)
-			)
-		))
+	)
 	(symbol
 		(lib_id "Connector_Generic:Conn_01x04")
@@
 			)
 		)
+		(property "LCSC" "C425129"
+			(at 59.69 90.17 0)
+			(hide yes)
+			(effects
+				(font
+					(size 1.27 1.27)
+				)
+			)
+		)
+		(property "MPN" "AYF530435"
+			(at 59.69 90.17 0)
+			(hide yes)
+			(effects
+				(font
+					(size 1.27 1.27)
+				)
+			)
+		)
+		(property "Note" "Encoder FFC leaf2"
+			(at 59.69 90.17 0)
+			(hide yes)
+			(effects
+				(font
+					(size 1.27 1.27)
+				)
+			)
+		)
 		(instances
 			(project "Connectors"
@@
 			)
 		)
-		(property "LCSC" "C425129"
-			(at 59.69 90.17 0)
-			(hide yes)
-			(effects
-				(font
-					(size 1.27 1.27)
-				)
-			)
-		)
-		(property "MPN" "AYF530435"
-			(at 59.69 90.17 0)
-			(hide yes)
-			(effects
-				(font
-					(size 1.27 1.27)
-				)
-			)
-		)
-		(property "Note" "Encoder FFC leaf2"
-			(at 59.69 90.17 0)
-			(hide yes)
-			(effects
-				(font
-					(size 1.27 1.27)
-				)
-			)
-		))
+	)
 	(symbol
 		(lib_id "Connector_Generic:Conn_01x04")
@@
 			)
 		)
+		(property "LCSC" "C425129"
+			(at 59.69 129.54 0)
+			(hide yes)
+			(effects
+				(font
+					(size 1.27 1.27)
+				)
+			)
+		)
+		(property "MPN" "AYF530435"
+			(at 59.69 129.54 0)
+			(hide yes)
+			(effects
+				(font
+					(size 1.27 1.27)
+				)
+			)
+		)
+		(property "Note" "Encoder FFC leaf3"
+			(at 59.69 129.54 0)
+			(hide yes)
+			(effects
+				(font
+					(size 1.27 1.27)
+				)
+			)
+		)
 		(instances
 			(project "Connectors"
@@
 			)
 		)
-		(property "LCSC" "C425129"
-			(at 59.69 129.54 0)
-			(hide yes)
-			(effects
-				(font
-					(size 1.27 1.27)
-				)
-			)
-		)
-		(property "MPN" "AYF530435"
-			(at 59.69 129.54 0)
-			(hide yes)
-			(effects
-				(font
-					(size 1.27 1.27)
-				)
-			)
-		)
-		(property "Note" "Encoder FFC leaf3"
-			(at 59.69 129.54 0)
-			(hide yes)
-			(effects
-				(font
-					(size 1.27 1.27)
-				)
-			)
-		))
+	)
 	(symbol
 		(lib_id "Connector_Generic:Conn_01x04")
@@
 			)
 		)
+		(property "LCSC" "C425129"
+			(at 59.69 170.18 0)
+			(hide yes)
+			(effects
+				(font
+					(size 1.27 1.27)
+				)
+			)
+		)
+		(property "MPN" "AYF530435"
+			(at 59.69 170.18 0)
+			(hide yes)
+			(effects
+				(font
+					(size 1.27 1.27)
+				)
+			)
+		)
+		(property "Note" "Encoder FFC leaf4"
+			(at 59.69 170.18 0)
+			(hide yes)
+			(effects
+				(font
+					(size 1.27 1.27)
+				)
+			)
+		)
 		(instances
 			(project "Connectors"
@@
 			)
 		)
-		(property "LCSC" "C425129"
-			(at 59.69 170.18 0)
-			(hide yes)
-			(effects
-				(font
-					(size 1.27 1.27)
-				)
-			)
-		)
-		(property "MPN" "AYF530435"
-			(at 59.69 170.18 0)
-			(hide yes)
-			(effects
-				(font
-					(size 1.27 1.27)
-				)
-			)
-		)
-		(property "Note" "Encoder FFC leaf4"
-			(at 59.69 170.18 0)
-			(hide yes)
-			(effects
-				(font
-					(size 1.27 1.27)
-				)
-			)
-		))
+	)
 	(symbol
 		(lib_id "Device:R")
@@
 			)
 		)
+		(property "Note" "Encoder SIG pull-up 10k to +3V3 - sensor output is open-drain; not optional (vault Encoder Interface)"
+			(at 100.33 44.45 0)
+			(hide yes)
+			(effects
+				(font
+					(size 1.27 1.27)
+				)
+			)
+		)
 		(instances
 			(project "Connectors"
@@
 			)
 		)
-		(property "Note" "Encoder SIG pull-up 10k to +3V3 - sensor output is open-drain; not optional (vault Encoder Interface)"
-			(at 100.33 44.45 0)
-			(hide yes)
-			(effects
-				(font
-					(size 1.27 1.27)
-				)
-			)
-		))
+	)
 	(symbol
 		(lib_id "Device:R")
@@
 	(symbol
 		(lib_id "power:GND")
-		(at 52.07 180.34 0)
+		(at 44.45 49.53 90)
 		(unit 1)
 		(in_bom yes)
@@
 		(dnp no)
 		(property "Reference" "#PWR002"
-			(at 52.07 186.69 0)
+			(at 50.8 49.53 0)
 			(hide yes)
 			(effects
@@
 		)
 		(property "Value" "GND"
-			(at 52.07 184.15 0)
+			(at 48.26 49.53 0)
 			(effects
 				(font
@@
 		)
 		(property "Footprint" ""
-			(at 52.07 180.34 0)
+			(at 44.45 49.53 0)
 			(hide yes)
 			(effects
@@
 		)
 		(property "Datasheet" ""
-			(at 52.07 180.34 0)
+			(at 44.45 49.53 0)
 			(hide yes)
 			(effects
@@
 					(reference "#PWR002")
 					(unit 1)
-				)
-			)
-			(project "MC3_COL_MAIN_V1.0"
-				(path "/7d5f4202-d55e-4c7b-a2df-dd599db38e48/d4085ee5-bdee-4718-a003-bbbd9ab9f320"
-					(reference "#PWR002")
-					(unit 1)

Commit message: Schematic annotated in eeschema (per-instance references for the 4 channel sheets); user review OK
Co-Authored-By: Claude Fable 5 <noreply@anthropic.com>
Parts:
- renumbered J4 to J3, J5 to J4, J6 to J5, J7 to J6, R30 to R6, R31 to R7, R32 to R8, R33 to R9

Commit message: Schematic re-annotated in eeschema after yaw channel + strap pull-ups
Co-Authored-By: Claude Fable 5 <noreply@anthropic.com>
Parts:
- renumbered R6 to R10, R7 to R11, R8 to R12, R9 to R13
Changed lines of the file:
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@@
 		(in_pos_files yes)
 		(dnp no)
-		(property "Reference" "R7"
+		(property "Reference" "R11"
 			(at 102.362 85.09 90)
 			(show_name no)
@@
 			(project "MC3_COL_MAIN_V1.0"
 				(path "/7d5f4202-d55e-4c7b-a2df-dd599db38e48/d4085ee5-bdee-4718-a003-bbbd9ab9f320"
-					(reference "R7")
+					(reference "R11")
 					(unit 1)
 				)
@@
 		(in_pos_files yes)
 		(dnp no)
-		(property "Reference" "R9"
+		(property "Reference" "R13"
 			(at 102.362 165.1 90)
 			(show_name no)
@@
 			(project "MC3_COL_MAIN_V1.0"
 				(path "/7d5f4202-d55e-4c7b-a2df-dd599db38e48/d4085ee5-bdee-4718-a003-bbbd9ab9f320"
-					(reference "R9")
+					(reference "R13")
 					(unit 1)
 				)
@@
 		(in_pos_files yes)
 		(dnp no)
-		(property "Reference" "R6"
+		(property "Reference" "R10"
 			(at 102.362 44.45 90)
 			(show_name no)
@@
 			(project "MC3_COL_MAIN_V1.0"
 				(path "/7d5f4202-d55e-4c7b-a2df-dd599db38e48/d4085ee5-bdee-4718-a003-bbbd9ab9f320"
-					(reference "R6")
+					(reference "R10")
 					(unit 1)
 				)
@@
 		(in_pos_files yes)
 		(dnp no)
-		(property "Reference" "R8"
+		(property "Reference" "R12"
 			(at 102.362 124.46 90)
 			(show_name no)
@@
 			(project "MC3_COL_MAIN_V1.0"
 				(path "/7d5f4202-d55e-4c7b-a2df-dd599db38e48/d4085ee5-bdee-4718-a003-bbbd9ab9f320"
-					(reference "R8")
-					(unit 1)
-				)
+					(reference "R12")
+					(unit 1)
+				)

Commit message: Design review changes: HSE caps 33pF, R_IPROPI 6.8k (1.99 A trip), VM bulk, sensor rail filter, input fuse+TVS, NRST cap, 6-pin SWD with SWO, VDDA ferrite, LEDs, test points, tantalum LDO cap
- MCU: C6/C10 18pF -> 33pF (X32258MSB4SI is CL=20pF); C60 100nF on NRST; J2 -> Conn_01x06
  (+NRST, +SWO on PB3); VDDA split from +3V3 through FB60 + PWR_FLAG; heartbeat LED D60/R60
  on PA5, power LED D61/R61; test points TP60-64 (+3V3, SCL, SDA, IPROPI_leaf1, GND)
- Power: J1 -> VIN_PAD -> F60 polyfuse -> VIN_PROT; D62 SMAJ5.0A TVS VIN_PROT-GND; C61/C62
  2x22uF VM bulk; TP65 VM, TP66 VIN_PROT; C2 LDO output cap -> tantalum 22uF 10V (C_Polarized,
  CP_EIA-3216-18)
- Connectors: FFC VIN now VSENS = VM through FB61 + C63 4.7uF
- MotorChannel: R_IPROPI 8.45k -> 6.8k (I_TRIP = 3.3/(6.8k*244uA/A) = 1.99 A)
- Library: stock L_0603, D_SMA, Fuse_1206, CP_EIA-3216-18, TestPoint_Pad_1.0x1.0mm, LED_0603,
  PinHeader_1x06 footprints copied in
- ERC 0 errors (same_local_global_label warnings only); netlist walked

Co-Authored-By: Claude Fable 5 <noreply@anthropic.com>
Parts:
- added C63: 4.7uF, MC3_COL_MAIN:C_0603_1608Metric, symbol Device:C
- added FB61: 600R@100MHz, MC3_COL_MAIN:L_0603_1608Metric, symbol Device:FerriteBead
Connections:
- net GND: now also C63.2
- net VM: now also FB61.1; no longer J3.1 (Pin_1), J4.1 (Pin_1), J5.1 (Pin_1), J6.1 (Pin_1)
- new net VSENS: C63.1, FB61.2, J3.1 (Pin_1), J4.1 (Pin_1), J5.1 (Pin_1), J6.1 (Pin_1)
Other:
- note added: "Review 2026-08-22: FFC VIN now from VSENS = VM filtered by FB61 + C63."

Commit message: LCSC/MPN fields on every support part (verified against the JLCPCB DB); R_IPROPI 6.8k = C93940; polyfuse 1206L200/12NR; MIGRATION register
Co-Authored-By: Claude Fable 5 <noreply@anthropic.com>
Parts:
- C63: LCSC (none) -> C19666; MPN (none) -> CL10A475KO8NNNC
- FB61: LCSC (none) -> C1002; MPN (none) -> GZ1608D601TF
- R10, R11, R12, R13: LCSC (none) -> C25744; MPN (none) -> 0402WGF1002TCE
Changed lines of the file:
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@@
 			)
 		)
-	)
+		(property "LCSC" "C25744"
+			(at 100.33 85.09 0)
+			(hide yes)
+			(effects
+				(font
+					(size 1.27 1.27)
+				)
+			)
+		)
+		(property "MPN" "0402WGF1002TCE"
+			(at 100.33 85.09 0)
+			(hide yes)
+			(effects
+				(font
+					(size 1.27 1.27)
+				)
+			)
+		))
 	(symbol
 		(lib_id "Device:R")
@@
 			)
 		)
-	)
+		(property "LCSC" "C25744"
+			(at 100.33 165.1 0)
+			(hide yes)
+			(effects
+				(font
+					(size 1.27 1.27)
+				)
+			)
+		)
+		(property "MPN" "0402WGF1002TCE"
+			(at 100.33 165.1 0)
+			(hide yes)
+			(effects
+				(font
+					(size 1.27 1.27)
+				)
+			)
+		))
 	(symbol
 		(lib_id "Connector_Generic:Conn_01x04")
@@
 			)
 		)
-	)
+		(property "LCSC" "C25744"
+			(at 100.33 44.45 0)
+			(hide yes)
+			(effects
+				(font
+					(size 1.27 1.27)
+				)
+			)
+		)
+		(property "MPN" "0402WGF1002TCE"
+			(at 100.33 44.45 0)
+			(hide yes)
+			(effects
+				(font
+					(size 1.27 1.27)
+				)
+			)
+		))
 	(symbol
 		(lib_id "Device:R")
@@
 			)
 		)
-	)
+		(property "LCSC" "C25744"
+			(at 100.33 124.46 0)
+			(hide yes)
+			(effects
+				(font
+					(size 1.27 1.27)
+				)
+			)
+		)
+		(property "MPN" "0402WGF1002TCE"
+			(at 100.33 124.46 0)
+			(hide yes)
+			(effects
+				(font
+					(size 1.27 1.27)
+				)
+			)
+		))
 	(symbol
 		(lib_id "Device:FerriteBead")
@@
 		)
 		(property "Note" "Sensor supply filter: VM -> ferrite 600R@100MHz -> VSENS (+4.7uF) feeding all four FFC VIN pins; keeps bridge PWM ripple off the LX34311 rail (review item 4). LCSC TBD"
+			(at 120.65 55.88 0)
+			(hide yes)
+			(effects
+				(font
+					(size 1.27 1.27)
+				)
+			)
+		)
+		(property "LCSC" "C1002"
+			(at 120.65 55.88 0)
+			(hide yes)
+			(effects
+				(font
+					(size 1.27 1.27)
+				)
+			)
+		)
+		(property "MPN" "GZ1608D601TF"
 			(at 120.65 55.88 0)
 			(hide yes)
@@
 			(at 130.81 55.88 0)
 			(hide yes)
+			(effects
+				(font
+					(size 1.27 1.27)
+				)
+			)
+		)
+		(property "LCSC" "C19666"
+			(at 130.81 55.88 0)
+			(hide yes)
+			(effects
+				(font
+					(size 1.27 1.27)
+				)
+			)
+		)
+		(property "MPN" "CL10A475KO8NNNC"
+			(at 130.81 55.88 0)
+			(hide yes)

Commit message: MCU -> STM32F412RET6 (pin-identical, adds bxCAN); CAN sheet: TJA1051T/3, split termination + jumper, PESD1CAN, CANH/CANL/GND pads
- MCU: U2 symbol MC3_COL_MAIN:STM32F412RET6 (same pin map as the F411), LCSC C89374; CAN1_RX PA11,
  CAN1_TX PA12; RC_OUT_leaf4 moved PA11 -> PB14
- CAN.kicad_sch (root sheet 'CAN'): U70 TJA1051T/3 (C38695) VCC from VM via FB62 + C70/C71,
  VIO +3V3, S low; JP70 solder jumper (bridged) -> R70/R71 62R split termination with C72 4.7nF;
  D70 PESD1CAN (C15771); J70 3 bare pads CANH/CANL/GND (new footprint SolderPads_3x)
- Library: STM32F412RET6 symbol; SolderPads_3x_2.2x1.4mm_P2.6mm, SOT-23, SolderJumper-2 footprints
- ERC 0 errors; netlist checked

Co-Authored-By: Claude Fable 5 <noreply@anthropic.com>
Parts:
- renumbered C63 to C17, FB61 to FB2, R10 to R12, R11 to R13, R12 to R14, R13 to R15

Commit message: Vault: COTS records for the CAN transceiver and encoder FFC; CAN decision and MCU Pinout updated
In the design wiki:
- COL-COTS-0030 TJA1051T/3. The /3 suffix is the reason for the part - separate
  VIO pin, so the bus runs at 5 V and the logic at 3.3 V with no level shifter.
  Flags that VCC comes off the motor rail through a bead, which depends on the
  still-unspecified machine supply being 5 V.
- COL-COTS-0031 Panasonic AYF530435. This one had been deliberately skipped as a
  "support part", which was the wrong call: it is a mechanical interface whose
  retention is a known risk - no solder tabs, four 0.5 mm joints taking the
  lever force, 20 mating cycles, on a board that rotates.
- Control Electronics: the control-link open item is resolved to CAN, recorded
  with why (Monoblock bus, differential in a motor enclosure, USB-CAN on the
  bench) and that it forced the MCU swap. Supply rail stays open; CAN added as
  decided-but-uncharacterized. The I2C open item now carries the 70 pF estimate.
- MCU Pinout: now the F412, with a table of the three assignments that moved,
  I2C1 fixed on PB8/PB9, the bus-capacitance working, and USB marked foreclosed
  since CAN took PA11/PA12.
- Datasheet index lists both new parts with their documents marked owed.

Repo side: U8 and J3-J6 now cite their records instead of "record owed" /
"no COTS record (support part)". Correcting those notes also caught a mislabel -
J4 and J5 both named the wrong leaf. ERC clean, 0 errors.

Co-Authored-By: Claude Opus 5 (1M context) <noreply@anthropic.com>
Parts:
- J3: COTS (none) -> COL-COTS-0031 (Panasonic AYF530435); Note Encoder FFC leaf1: 1 VIN(VM) 2 GND 3 SIG 4 spare. No COTS r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 -> Encoder FFC leaf1: 1 VIN(VM) 2 GND 3 SIG 4 spare. Vault: CO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
- J4: COTS (none) -> COL-COTS-0031 (Panasonic AYF530435); Note Encoder FFC leaf2 -> Encoder FFC leaf2: 1 VIN(VM) 2 GND 3 SIG 4 spare. Vault: CO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
- J5: COTS (none) -> COL-COTS-0031 (Panasonic AYF530435); Note Encoder FFC leaf3 -> Encoder FFC leaf3: 1 VIN(VM) 2 GND 3 SIG 4 spare. Vault: CO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
- J6: COTS (none) -> COL-COTS-0031 (Panasonic AYF530435); Note Encoder FFC leaf4 -> Encoder FFC leaf4: 1 VIN(VM) 2 GND 3 SIG 4 spare. Vault: CO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
Changed lines of the file:
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@@
 			)
 		)
-		(property "Note" "Encoder FFC leaf1: 1 VIN(VM) 2 GND 3 SIG 4 spare. No COTS record (support part) - vault Connectors / Encoder Interface"
+		(property "Note" "Encoder FFC leaf1: 1 VIN(VM) 2 GND 3 SIG 4 spare. Vault: COL-COTS-0031, Connectors / Encoder Interface. Right-angle SMD, no solder tabs - the four 0.5mm joints are the only mechanical attachment; footprint mech pads are netless and should be tied to GND"
 			(at 59.69 49.53 0)
 			(hide yes)
@@
 			)
 		)
-	)
+		(property "COTS" "COL-COTS-0031 (Panasonic AYF530435)"
+			(at 59.69 49.53 0)
+			(hide yes)
+			(effects
+				(font
+					(size 1.27 1.27)
+				)
+			)
+		))
 	(symbol
 		(lib_id "power:GND")
@@
 			)
 		)
-		(property "Note" "Encoder FFC leaf4"
+		(property "Note" "Encoder FFC leaf4: 1 VIN(VM) 2 GND 3 SIG 4 spare. Vault: COL-COTS-0031, Connectors / Encoder Interface"
 			(at 59.69 170.18 0)
 			(hide yes)
@@
 			)
 		)
-	)
+		(property "COTS" "COL-COTS-0031 (Panasonic AYF530435)"
+			(at 59.69 170.18 0)
+			(hide yes)
+			(effects
+				(font
+					(size 1.27 1.27)
+				)
+			)
+		))
 	(symbol
 		(lib_id "power:+3V3")
@@
 			)
 		)
-		(property "Note" "Encoder FFC leaf2"
+		(property "Note" "Encoder FFC leaf2: 1 VIN(VM) 2 GND 3 SIG 4 spare. Vault: COL-COTS-0031, Connectors / Encoder Interface"
 			(at 59.69 90.17 0)
 			(hide yes)
@@
 			)
 		)
-	)
+		(property "COTS" "COL-COTS-0031 (Panasonic AYF530435)"
+			(at 59.69 90.17 0)
+			(hide yes)
+			(effects
+				(font
+					(size 1.27 1.27)
+				)
+			)
+		))
 	(symbol
 		(lib_id "Connector_Generic:Conn_01x04")
@@
 			)
 		)
-		(property "Note" "Encoder FFC leaf3"
+		(property "Note" "Encoder FFC leaf3: 1 VIN(VM) 2 GND 3 SIG 4 spare. Vault: COL-COTS-0031, Connectors / Encoder Interface"
 			(at 59.69 129.54 0)
 			(hide yes)
@@
 			)
 		)
-	)
+		(property "COTS" "COL-COTS-0031 (Panasonic AYF530435)"
+			(at 59.69 129.54 0)
+			(hide yes)
+			(effects
+				(font
+					(size 1.27 1.27)
+				)
+			)
+		))
 	(symbol
 		(lib_id "Device:FerriteBead")
