File: boards/MC3_COL_MAIN_V1.0/CAN.kicad_sch (KiCad schematic)
At the start: 10 parts, among them J12 CAN, U8 TJA1051T/3

Commit message: Vault: COTS records for the CAN transceiver and encoder FFC; CAN decision and MCU Pinout updated
In the design wiki:
- COL-COTS-0030 TJA1051T/3. The /3 suffix is the reason for the part - separate
  VIO pin, so the bus runs at 5 V and the logic at 3.3 V with no level shifter.
  Flags that VCC comes off the motor rail through a bead, which depends on the
  still-unspecified machine supply being 5 V.
- COL-COTS-0031 Panasonic AYF530435. This one had been deliberately skipped as a
  "support part", which was the wrong call: it is a mechanical interface whose
  retention is a known risk - no solder tabs, four 0.5 mm joints taking the
  lever force, 20 mating cycles, on a board that rotates.
- Control Electronics: the control-link open item is resolved to CAN, recorded
  with why (Monoblock bus, differential in a motor enclosure, USB-CAN on the
  bench) and that it forced the MCU swap. Supply rail stays open; CAN added as
  decided-but-uncharacterized. The I2C open item now carries the 70 pF estimate.
- MCU Pinout: now the F412, with a table of the three assignments that moved,
  I2C1 fixed on PB8/PB9, the bus-capacitance working, and USB marked foreclosed
  since CAN took PA11/PA12.
- Datasheet index lists both new parts with their documents marked owed.

Repo side: U8 and J3-J6 now cite their records instead of "record owed" /
"no COTS record (support part)". Correcting those notes also caught a mislabel -
J4 and J5 both named the wrong leaf. ERC clean, 0 errors.

Co-Authored-By: Claude Opus 5 (1M context) <noreply@anthropic.com>
Parts:
- U8: COTS COL-COTS-TBD (engineering part - CAN transceiver, record ow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 -> COL-COTS-0030 (TJA1051T/3 CAN transceiver)
Changed lines of the file:
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@@
 			)
 		)
-		(property "COTS" "COL-COTS-TBD (engineering part - CAN transceiver, record owed)"
+		(property "COTS" "COL-COTS-0030 (TJA1051T/3 CAN transceiver)"
 			(at 100.33 80.01 0)
 			(hide yes)

Commit message: Review fixes applied (C21, C37 order, stitching vias) + review-driven adds: 5x 1nF IPROPI ADC filters (C38-42, C1523), U8 VIO 100nF (C43), 3x M2.5 NPTH mounting holes (H1-3) - caps placed unwired, user wires; holes placed in layout by user
Co-Authored-By: Claude Fable 5 <noreply@anthropic.com>
Parts:
- added C43: 100nF, MC3_COL_MAIN:C_0402_1005Metric, symbol Device:C
Changed lines of the file:
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@@
 	(generator_version "10.0")
 	(paper "A4")
-	(text "CAN - machine control link (decision 2026-08-22; vault Control Electronics open item). STM32F412 CAN1 (PA11 RX / PA12 TX) -> TJA1051T/3 -> split termination (2x62R + 4.7nF, solder-jumper JP70 bridged) + PESD1CAN -> pads CANH/CANL/GND. Classic CAN 500 kbit/s. Layout: CANH/CANL as a tight pair, transceiver and termination next to the pads, D70 nearest the pads."
-		(exclude_from_sim no)
-		(at 30 40 0)
-		(effects
-			(font
-				(size 1.5 1.5)
-			)
-		)
-	)
 	(wire
 		(pts
-			(xy 87.63 82.55) (xy 85.09 82.55)
+			(xy 87.63 82.55)
+			(xy 85.09 82.55)
 		)
 		(stroke
@@
 	(wire
 		(pts
-			(xy 87.63 77.47) (xy 85.09 77.47)
+			(xy 87.63 77.47)
+			(xy 85.09 77.47)
 		)
 		(stroke
@@
 	(wire
 		(pts
-			(xy 87.63 74.93) (xy 85.09 74.93)
+			(xy 87.63 74.93)
+			(xy 85.09 74.93)
 		)
 		(stroke
@@
 	(wire
 		(pts
-			(xy 60.96 57.15) (xy 60.96 54.61)
+			(xy 60.96 57.15)
+			(xy 60.96 54.61)
 		)
 		(stroke
 			(width 0)
 			(type default)
+		)
+	)
+	(text "CAN - machine control link (decision 2026-08-22; vault Control Electronics open item). STM32F412 CAN1 (PA11 RX / PA12 TX) -> TJA1051T/3 -> split termination (2x62R + 4.7nF, solder-jumper JP70 bridged) + PESD1CAN -> pads CANH/CANL/GND. Classic CAN 500 kbit/s. Layout: CANH/CANL as a tight pair, transceiver and termination next to the pads, D70 nearest the pads."
+		(at 30 40 0)
+		(effects
+			(font
+				(size 1.5 1.5)
+			)
 		)
 	)
@@
 		(at 135.89 88.9 90)
 		(unit 1)
-		(body_style 1)
 		(exclude_from_sim no)
 		(in_bom yes)
 		(on_board yes)
-		(in_pos_files yes)
 		(dnp no)
 		(property "Reference" "R32"
@@
 			)
 		)
+		(body_style 1)
+		(in_pos_files yes)
 		(pin "1"
 		)
@@
 		(at 165.1 80.01 0)
 		(unit 1)
-		(body_style 1)
 		(exclude_from_sim no)
 		(in_bom yes)
 		(on_board yes)
-		(in_pos_files yes)
 		(dnp no)
 		(property "Reference" "J12"
@@
 			)
 		)
+		(body_style 1)
+		(in_pos_files yes)
 		(pin "1"
 		)
@@
 		(at 71.12 66.04 0)
 		(unit 1)
-		(body_style 1)
 		(exclude_from_sim no)
 		(in_bom yes)
 		(on_board yes)
-		(in_pos_files yes)
 		(dnp no)
 		(property "Reference" "C28"
@@
 			)
 		)
+		(body_style 1)
+		(in_pos_files yes)
 		(pin "1"
 		)
@@
 		(at 125.73 100.33 0)
 		(unit 1)
-		(body_style 1)
 		(exclude_from_sim no)
 		(in_bom yes)
 		(on_board yes)
-		(in_pos_files yes)
 		(dnp no)
 		(property "Reference" "D4"
@@
 			)
 		)
+		(body_style 1)
+		(in_pos_files yes)
 		(pin "3"
 		)
@@
 		(at 78.74 66.04 0)
 		(unit 1)
-		(body_style 1)
 		(exclude_from_sim no)
 		(in_bom yes)
 		(on_board yes)
-		(in_pos_files yes)
 		(dnp no)
 		(property "Reference" "C29"
@@
 			)
 		)
+		(body_style 1)
+		(in_pos_files yes)
 		(pin "1"
 		)
@@
 		(at 125.73 71.12 0)
 		(unit 1)
-		(body_style 1)
 		(exclude_from_sim no)
 		(in_bom yes)
 		(on_board yes)
-		(in_pos_files yes)
 		(dnp no)
 		(property "Reference" "JP1"
@@
 			)
 		)
+		(body_style 1)
+		(in_pos_files yes)
 		(pin "1"
 		)
@@
 		(at 60.96 60.96 0)
 		(unit 1)
-		(body_style 1)
 		(exclude_from_sim no)
 		(in_bom yes)
 		(on_board yes)
-		(in_pos_files yes)
 		(dnp no)
 		(property "Reference" "FB3"
@@
 			)
 		)
+		(body_style 1)
+		(in_pos_files yes)
 		(pin "1"
 		)
@@
 		(at 135.89 71.12 90)
 		(unit 1)
-		(body_style 1)
 		(exclude_from_sim no)
 		(in_bom yes)
 		(on_board yes)
-		(in_pos_files yes)
 		(dnp no)
 		(property "Reference" "R31"
@@
 			)
 		)
+		(body_style 1)
+		(in_pos_files yes)
 		(pin "1"
 		)
@@
 		(at 146.05 80.01 0)
 		(unit 1)
-		(body_style 1)
 		(exclude_from_sim no)
 		(in_bom yes)
 		(on_board yes)
-		(in_pos_files yes)
 		(dnp no)
 		(property "Reference" "C30"
@@
 			)
 		)
+		(body_style 1)
+		(in_pos_files yes)
 		(pin "1"
 		)
@@
 		(at 100.33 90.17 0)
 		(unit 1)
-		(body_style 1)
 		(exclude_from_sim no)
 		(in_bom yes)
 		(on_board yes)
-		(in_pos_files yes)
 		(dnp no)
 		(property "Reference" "#PWR022"
@@
 			)
 		)
+		(body_style 1)
+		(in_pos_files yes)
 		(pin "1"
 		)
@@
 		(at 100.33 80.01 0)
 		(unit 1)
-		(body_style 1)
 		(exclude_from_sim no)
 		(in_bom yes)
 		(on_board yes)
-		(in_pos_files yes)
 		(dnp no)
 		(property "Reference" "U8"
@@
 			)
 		)
+		(body_style 1)
+		(in_pos_files yes)
 		(pin "1"
 		)
@@
 		(at 60.96 64.77 180)
 		(unit 1)
-		(body_style 1)
 		(exclude_from_sim no)
 		(in_bom yes)
 		(on_board yes)
-		(in_pos_files yes)
 		(dnp no)
 		(property "Reference" "#PWR021"
@@
 			)
 		)
+		(body_style 1)
+		(in_pos_files yes)
 		(pin "1"
 		)
@@
 		)
 	)
+	(symbol
+		(lib_id "Device:C")
+		(at 71.12 110.49 0)
+		(unit 1)
+		(in_bom yes)
+		(on_board yes)
+		(dnp no)
+		(property "Reference" "C43"
+			(at 71.755 107.95 0)
+			(effects
+				(font
+					(size 1.27 1.27)
+				)
+				(justify left)
+			)
+		)
+		(property "Value" "100nF"
+			(at 71.755 113.03 0)
+			(effects
+				(font
+					(size 1.27 1.27)
+				)
+				(justify left)
+			)
+		)
+		(property "Footprint" "MC3_COL_MAIN:C_0402_1005Metric"
+			(at 71.12 110.49 0)
+			(hide yes)
+			(effects
+				(font
+					(size 1.27 1.27)
+				)
+			)
+		)
+		(property "Datasheet" ""
+			(at 71.12 110.49 0)
+			(hide yes)
+			(effects
+				(font
+					(size 1.27 1.27)
+				)
+			)
+		)
+		(instances
+			(project "MC3_COL_MAIN_V1.0"
+				(path "/7d5f4202-d55e-4c7b-a2df-dd599db38e48/d53768a6-e0ca-46e0-8386-8014881aa541"
+					(reference "C43")
+					(unit 1)
+				)
+			)
+		)
+		(property "LCSC" "C1525"
+			(at 71.12 110.49 0)
+			(hide yes)
+			(effects
+				(font
+					(size 1.27 1.27)
+				)
+			)
+		)
+		(property "Note" "U8 VIO (pin 5) local decoupling - place within 4 mm of pin 5; wire pin1 to +3V3, pin2 to GND"
+			(at 71.12 110.49 0)
+			(hide yes)
+			(effects
+				(font
+					(size 1.27 1.27)
+				)
+			)
+		))
 )

Commit message: Wire the review caps: C38-42 onto IPROPI_* (global labels) + GND, C43 onto +3V3/GND; power refs #PWR0115-0121
Co-Authored-By: Claude Fable 5 <noreply@anthropic.com>
Connections:
- net +3V3: now also C43.1
- net GND: now also C43.2
Changed lines of the file:
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@@
-			)
-		)
-		(instances
-			(project "MC3_COL_MAIN_V1.0"
-				(path "/7d5f4202-d55e-4c7b-a2df-dd599db38e48/d53768a6-e0ca-46e0-8386-8014881aa541"
-					(reference "C43")
-					(unit 1)
-				)
 			)
 		)
@@
 				)
 			)
-		))
+		)
+		(instances
+			(project "MC3_COL_MAIN_V1.0"
+				(path "/7d5f4202-d55e-4c7b-a2df-dd599db38e48/d53768a6-e0ca-46e0-8386-8014881aa541"
+					(reference "C43")
+					(unit 1)
+				)
+			)
+		)
+	)
+	(symbol
+		(lib_id "power:+3V3")
+		(at 71.12 106.68 0)
+		(unit 1)
+		(in_bom yes)
+		(on_board yes)
+		(dnp no)
+		(property "Reference" "#PWR0120"
+			(at 71.12 110.49 0)
+			(hide yes)
+			(effects
+				(font
+					(size 1.27 1.27)
+				)
+			)
+		)
+		(property "Value" "+3V3"
+			(at 71.12 103.124 0)
+			(effects
+				(font
+					(size 1.27 1.27)
+				)
+			)
+		)
+		(property "Footprint" ""
+			(at 71.12 106.68 0)
+			(hide yes)
+			(effects
+				(font
+					(size 1.27 1.27)
+				)
+			)
+		)
+		(property "Datasheet" ""
+			(at 71.12 106.68 0)
+			(hide yes)
+			(effects
+				(font
+					(size 1.27 1.27)
+				)
+			)
+		)
+		(instances
+			(project "CAN"
+				(path "/3d434ce1-889d-46d1-8950-1c686d039f9f"
+					(reference "#PWR0120")
+					(unit 1)
+				)
+			)
+		)
+	)
+	(symbol
+		(lib_id "power:GND")
+		(at 71.12 114.3 0)
+		(unit 1)
+		(in_bom yes)
+		(on_board yes)
+		(dnp no)
+		(property "Reference" "#PWR0121"
+			(at 71.12 120.65 0)
+			(hide yes)
+			(effects
+				(font
+					(size 1.27 1.27)
+				)
+			)
+		)
+		(property "Value" "GND"
+			(at 71.12 118.11 0)
+			(effects
+				(font
+					(size 1.27 1.27)
+				)
+			)
+		)
+		(property "Footprint" ""
+			(at 71.12 114.3 0)
+			(hide yes)
+			(effects
+				(font
+					(size 1.27 1.27)
+				)
+			)
+		)
+		(property "Datasheet" ""
+			(at 71.12 114.3 0)
+			(hide yes)
+			(effects
+				(font
+					(size 1.27 1.27)
+				)
+			)
+		)
+		(instances
+			(project "CAN"
+				(path "/3d434ce1-889d-46d1-8950-1c686d039f9f"
+					(reference "#PWR0121")
+					(unit 1)
+				)
+			)
+		)
+	)
 )
