File: boards/MC3_COL_MAIN_V1.0/MC3_COL_MAIN_V1.0.kicad_sch (KiCad schematic)
At the start: 4 parts

Commit message: User: re-annotated schematic (CAN/F412 parts), drill/place + grid origin at (100,100) saved in the board
Co-Authored-By: Claude Fable 5 <noreply@anthropic.com>
Changed lines of the file:
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@@
+	)
+	(sheet
+		(at 223.52 19.05)
+		(size 45.72 25.4)
+		(exclude_from_sim no)
+		(in_bom yes)
+		(on_board yes)
+		(dnp no)
+		(fields_autoplaced yes)
+		(stroke
+			(width 0.1524)
+			(type solid)
+		)
+		(fill
+			(color 0 0 0 0)
+		)
+		(property "Sheetname" "CAN"
+			(at 223.52 18.415 0)
+			(show_name no)
+			(do_not_autoplace no)
+			(effects
+				(font
+					(size 1.27 1.27)
+				)
+				(justify left bottom)
+			)
+		)
+		(property "Sheetfile" "CAN.kicad_sch"
+			(at 223.52 45.085 0)
+			(show_name no)
+			(do_not_autoplace no)
+			(effects
+				(font
+					(size 1.27 1.27)
+				)
+				(justify left top)
+			)
+		)
+		(instances
+			(project "MC3_COL_MAIN_V1.0"
+				(path "/7d5f4202-d55e-4c7b-a2df-dd599db38e48"
+					(page "10")
+				)
+			)
+		)
 	)
 	(sheet
@@
 		)
 	)
-	(sheet
-    (at 160.02 140.97)
-    (size 45.72 25.4)
-    (fields_autoplaced yes)
-    (stroke (width 0.1524) (type solid))
-    (fill (color 0 0 0 0.0))
-    (property "Sheetname" "CAN"
-      (at 160.02 140.335 0)
-      (effects (font (size 1.27 1.27)) (justify left bottom))
-    )
-    (property "Sheetfile" "CAN.kicad_sch"
-      (at 160.02 167.005 0)
-      (effects (font (size 1.27 1.27)) (justify left top))
-    )
-    (instances
-      (project "MC3_COL_MAIN_V1.0"
-        (path "/7d5f4202-d55e-4c7b-a2df-dd599db38e48" (page "10"))
-      )
-    )
-  )
 	(sheet_instances
 		(path "/"

Commit message: Review fixes applied (C21, C37 order, stitching vias) + review-driven adds: 5x 1nF IPROPI ADC filters (C38-42, C1523), U8 VIO 100nF (C43), 3x M2.5 NPTH mounting holes (H1-3) - caps placed unwired, user wires; holes placed in layout by user
Co-Authored-By: Claude Fable 5 <noreply@anthropic.com>
Parts:
- added H1, H2, H3: M2.5, MC3_COL_MAIN:MountingHole_2.7mm_M2.5, symbol Mechanical:MountingHole

Commit message: Mounting holes H1-H3: M2.5 -> M2 (2.2mm NPTH) - user call, tight annulus
Co-Authored-By: Claude Fable 5 <noreply@anthropic.com>
Parts:
- H1, H2, H3: value M2.5 -> M2; footprint MC3_COL_MAIN:MountingHole_2.7mm_M2.5 -> MC3_COL_MAIN:MountingHole_2.2mm_M2; Note NPTH 2.7 mm clearance for M2.5, electrically isolated; 3x ~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 -> NPTH 2.2 mm clearance for M2, electrically isolated; 3x ~12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
Changed lines of the file:
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@@
 			)
 		)
-		(property "Value" "M2.5"
+		(property "Value" "M2"
 			(at 40.64 107.315 0)
 			(effects
@@
 			)
 		)
-		(property "Footprint" "MC3_COL_MAIN:MountingHole_2.7mm_M2.5"
+		(property "Footprint" "MC3_COL_MAIN:MountingHole_2.2mm_M2"
 			(at 40.64 110.49 0)
 			(hide yes)
@@
 			)
 		)
-		(property "Note" "NPTH 2.7 mm clearance for M2.5, electrically isolated; 3x ~120 deg apart, positions set in layout (board-to-frame spacing = the encoder gap, PARAM owed)"
+		(property "Note" "NPTH 2.2 mm clearance for M2, electrically isolated; 3x ~120 deg apart, positions set in layout (board-to-frame spacing = the encoder gap, PARAM owed)"
 			(at 40.64 110.49 0)
 			(hide yes)
@@
 			)
 		)
-		(property "Value" "M2.5"
+		(property "Value" "M2"
 			(at 53.34 107.315 0)
 			(effects
@@
 			)
 		)
-		(property "Footprint" "MC3_COL_MAIN:MountingHole_2.7mm_M2.5"
+		(property "Footprint" "MC3_COL_MAIN:MountingHole_2.2mm_M2"
 			(at 53.34 110.49 0)
 			(hide yes)
@@
 			)
 		)
-		(property "Note" "NPTH 2.7 mm clearance for M2.5, electrically isolated; 3x ~120 deg apart, positions set in layout (board-to-frame spacing = the encoder gap, PARAM owed)"
+		(property "Note" "NPTH 2.2 mm clearance for M2, electrically isolated; 3x ~120 deg apart, positions set in layout (board-to-frame spacing = the encoder gap, PARAM owed)"
 			(at 53.34 110.49 0)
 			(hide yes)
@@
 			)
 		)
-		(property "Value" "M2.5"
+		(property "Value" "M2"
 			(at 66.04 107.315 0)
 			(effects
@@
 			)
 		)
-		(property "Footprint" "MC3_COL_MAIN:MountingHole_2.7mm_M2.5"
+		(property "Footprint" "MC3_COL_MAIN:MountingHole_2.2mm_M2"
 			(at 66.04 110.49 0)
 			(hide yes)
@@
 			)
 		)
-		(property "Note" "NPTH 2.7 mm clearance for M2.5, electrically isolated; 3x ~120 deg apart, positions set in layout (board-to-frame spacing = the encoder gap, PARAM owed)"
+		(property "Note" "NPTH 2.2 mm clearance for M2, electrically isolated; 3x ~120 deg apart, positions set in layout (board-to-frame spacing = the encoder gap, PARAM owed)"
 			(at 66.04 110.49 0)
 			(hide yes)

Commit message: H4: pass-through slot placeholder (NPTH, user converts to oval + positions) - temporary yaw motor lead routing to the power/CAN pad area
Co-Authored-By: Claude Fable 5 <noreply@anthropic.com>
Parts:
- added H4: SLOT-PASSTHRU, MC3_COL_MAIN:SlotNPTH_PassThrough, symbol Mechanical:MountingHole
Changed lines of the file:
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@@
+	)
+	(symbol
+		(lib_id "Mechanical:MountingHole")
+		(at 66.04 110.49 0)
+		(unit 1)
+		(exclude_from_sim no)
+		(in_bom yes)
+		(on_board yes)
+		(dnp no)
+		(property "Reference" "H3"
+			(at 66.04 105.41 0)
+			(show_name no)
+			(do_not_autoplace no)
+			(effects
+				(font
+					(size 1.27 1.27)
+				)
+			)
+		)
+		(property "Value" "M2"
+			(at 66.04 107.315 0)
+			(show_name no)
+			(do_not_autoplace no)
+			(effects
+				(font
+					(size 1.27 1.27)
+				)
+			)
+		)
+		(property "Footprint" "MC3_COL_MAIN:MountingHole_2.2mm_M2"
+			(at 66.04 110.49 0)
+			(hide yes)
+			(show_name no)
+			(do_not_autoplace no)
+			(effects
+				(font
+					(size 1.27 1.27)
+				)
+			)
+		)
+		(property "Datasheet" ""
+			(at 66.04 110.49 0)
+			(hide yes)
+			(show_name no)
+			(do_not_autoplace no)
+			(effects
+				(font
+					(size 1.27 1.27)
+				)
+			)
+		)
+		(property "Description" ""
+			(at 66.04 110.49 0)
+			(show_name no)
+			(do_not_autoplace no)
+			(effects
+				(font
+					(size 1.27 1.27)
+				)
+			)
+		)
+		(property "Note" "NPTH 2.2 mm clearance for M2, electrically isolated; 3x ~120 deg apart, positions set in layout (board-to-frame spacing = the encoder gap, PARAM owed)"
+			(at 66.04 110.49 0)
+			(hide yes)
+			(show_name no)
+			(do_not_autoplace no)
+			(effects
+				(font
+					(size 1.27 1.27)
+				)
+			)
+		)
+		(body_style 1)
+		(in_pos_files yes)
+		(instances
+			(project "MC3_COL_MAIN_V1.0"
+				(path "/7d5f4202-d55e-4c7b-a2df-dd599db38e48"
+					(reference "H3")
+					(unit 1)
+				)
+			)
+		)
 	)
 	(symbol
@@
 	(symbol
 		(lib_id "Mechanical:MountingHole")
+		(at 53.34 110.49 0)
+		(unit 1)
+		(exclude_from_sim no)
+		(in_bom yes)
+		(on_board yes)
+		(dnp no)
+		(property "Reference" "H2"
+			(at 53.34 105.41 0)
+			(show_name no)
+			(do_not_autoplace no)
+			(effects
+				(font
+					(size 1.27 1.27)
+				)
+			)
+		)
+		(property "Value" "M2"
+			(at 53.34 107.315 0)
+			(show_name no)
+			(do_not_autoplace no)
+			(effects
+				(font
+					(size 1.27 1.27)
+				)
+			)
+		)
+		(property "Footprint" "MC3_COL_MAIN:MountingHole_2.2mm_M2"
+			(at 53.34 110.49 0)
+			(hide yes)
+			(show_name no)
+			(do_not_autoplace no)
+			(effects
+				(font
+					(size 1.27 1.27)
+				)
+			)
+		)
+		(property "Datasheet" ""
+			(at 53.34 110.49 0)
+			(hide yes)
+			(show_name no)
+			(do_not_autoplace no)
+			(effects
+				(font
+					(size 1.27 1.27)
+				)
+			)
+		)
+		(property "Description" ""
+			(at 53.34 110.49 0)
+			(show_name no)
+			(do_not_autoplace no)
+			(effects
+				(font
+					(size 1.27 1.27)
+				)
+			)
+		)
+		(property "Note" "NPTH 2.2 mm clearance for M2, electrically isolated; 3x ~120 deg apart, positions set in layout (board-to-frame spacing = the encoder gap, PARAM owed)"
+			(at 53.34 110.49 0)
+			(hide yes)
+			(show_name no)
+			(do_not_autoplace no)
+			(effects
+				(font
+					(size 1.27 1.27)
+				)
+			)
+		)
+		(body_style 1)
+		(in_pos_files yes)
+		(instances
+			(project "MC3_COL_MAIN_V1.0"
+				(path "/7d5f4202-d55e-4c7b-a2df-dd599db38e48"
+					(reference "H2")
+					(unit 1)
+				)
+			)
+		)
+	)
+	(symbol
+		(lib_id "Mechanical:MountingHole")
 		(at 40.64 110.49 0)
 		(unit 1)
+		(exclude_from_sim no)
 		(in_bom yes)
 		(on_board yes)
@@
 		(property "Reference" "H1"
 			(at 40.64 105.41 0)
+			(show_name no)
+			(do_not_autoplace no)
 			(effects
 				(font
@@
 		(property "Value" "M2"
 			(at 40.64 107.315 0)
+			(show_name no)
+			(do_not_autoplace no)
 			(effects
 				(font
@@
 			(at 40.64 110.49 0)
 			(hide yes)
+			(show_name no)
+			(do_not_autoplace no)
 			(effects
 				(font
@@
 			(at 40.64 110.49 0)
 			(hide yes)
+			(show_name no)
+			(do_not_autoplace no)
+			(effects
+				(font
+					(size 1.27 1.27)
+				)
+			)
+		)
+		(property "Description" ""
+			(at 40.64 110.49 0)
+			(show_name no)
+			(do_not_autoplace no)
 			(effects
 				(font
@@
 			(at 40.64 110.49 0)
 			(hide yes)
-			(effects
-				(font
-					(size 1.27 1.27)
-				)
-			)
-		)
+			(show_name no)
+			(do_not_autoplace no)
+			(effects
+				(font
+					(size 1.27 1.27)
+				)
+			)
+		)
+		(body_style 1)
+		(in_pos_files yes)
 		(instances
 			(project "MC3_COL_MAIN_V1.0"
@@
 	(symbol
 		(lib_id "Mechanical:MountingHole")
-		(at 53.34 110.49 0)
+		(at 78.74 110.49 0)
 		(unit 1)
 		(in_bom yes)
 		(on_board yes)
 		(dnp no)
-		(property "Reference" "H2"
-			(at 53.34 105.41 0)
-			(effects
-				(font
-					(size 1.27 1.27)
-				)
-			)
-		)
-		(property "Value" "M2"
-			(at 53.34 107.315 0)
-			(effects
-				(font
-					(size 1.27 1.27)
-				)
-			)
-		)
-		(property "Footprint" "MC3_COL_MAIN:MountingHole_2.2mm_M2"
-			(at 53.34 110.49 0)
+		(property "Reference" "H4"
+			(at 78.74 105.41 0)
+			(effects
+				(font
+					(size 1.27 1.27)
+				)
+			)
+		)
+		(property "Value" "SLOT-PASSTHRU"
+			(at 78.74 107.315 0)
+			(effects
+				(font
+					(size 1.27 1.27)
+				)
+			)
+		)
+		(property "Footprint" "MC3_COL_MAIN:SlotNPTH_PassThrough"
+			(at 78.74 110.49 0)
 			(hide yes)
 			(effects
@@
 		)
 		(property "Datasheet" ""
-			(at 53.34 110.49 0)
-			(hide yes)
-			(effects
-				(font
-					(size 1.27 1.27)
-				)
-			)
-		)
-		(property "Note" "NPTH 2.2 mm clearance for M2, electrically isolated; 3x ~120 deg apart, positions set in layout (board-to-frame spacing = the encoder gap, PARAM owed)"
-			(at 53.34 110.49 0)
+			(at 78.74 110.49 0)
 			(hide yes)
 			(effects
@@
 			(project "MC3_COL_MAIN_V1.0"
 				(path "/7d5f4202-d55e-4c7b-a2df-dd599db38e48"
-					(reference "H2")
+					(reference "H4")
 					(unit 1)
 				)
 			)
 		)
-	)
-	(symbol
-		(lib_id "Mechanical:MountingHole")
-		(at 66.04 110.49 0)
-		(unit 1)
-		(in_bom yes)
-		(on_board yes)
-		(dnp no)
-		(property "Reference" "H3"
-			(at 66.04 105.41 0)
-			(effects
-				(font
-					(size 1.27 1.27)
-				)
-			)
-		)
-		(property "Value" "M2"
-			(at 66.04 107.315 0)
-			(effects
-				(font
-					(size 1.27 1.27)
-				)
-			)
-		)
-		(property "Footprint" "MC3_COL_MAIN:MountingHole_2.2mm_M2"
-			(at 66.04 110.49 0)
-			(hide yes)
-			(effects
-				(font
-					(size 1.27 1.27)
-				)
-			)
-		)
-		(property "Datasheet" ""
-			(at 66.04 110.49 0)
-			(hide yes)
-			(effects
-				(font
-					(size 1.27 1.27)
-				)
-			)
-		)
-		(instances
-			(project "MC3_COL_MAIN_V1.0"
-				(path "/7d5f4202-d55e-4c7b-a2df-dd599db38e48"
-					(reference "H3")
-					(unit 1)
-				)
-			)
-		)
-		(property "Note" "NPTH 2.2 mm clearance for M2, electrically isolated; 3x ~120 deg apart, positions set in layout (board-to-frame spacing = the encoder gap, PARAM owed)"
-			(at 66.04 110.49 0)
-			(hide yes)
-			(effects
+		(property "Note" "PROVISIONAL - wire pass-through slot for temporarily routing the yaw motor leads to the power/CAN pad area on the back. Placeholder circular 2.5mm NPTH: in the footprint editor set Hole shape = Oval and tune size; position in layout. Delete when the yaw lead routing is permanent"
+			(at 78.74 110.49 0)
+			(hide yes)
+			(effects
