File: boards/MC3_COL_MAIN_V1.0/MC3_COL_MAIN_V1.0.kicad_sch (KiCad schematic)
At the start: 8 parts

Commit message: WIP checkpoint before LED chain (board session state as on disk)
Parts:
- added H4: M2, MC3_COL_MAIN:MountingHole_2.2mm_M2, symbol Mechanical:MountingHole
- renumbered H4 to H5
Other:
- moved on the sheet: H5
