File: boards/MC3_COL_MAIN_V1.0/_restore_backup_2026-08-22T14-11-53-608/Connectors.kicad_sch (KiCad schematic)
At the start: 10 parts, among them J12 CAN, U8 TJA1051T/3

Commit message: PCB placement pass 2: all five motor channels on one uniform pattern
User decision: drop the per-channel rotation. leaf3 (arranged by hand in the
GUI) is the pattern; leaf1, leaf2, leaf4 and yaw are now byte-identical copies
of its relative geometry at the same orientation - driver at -90, top row of
0402s at dy -3.5, 1 uF VM cap at (-3, +1), address straps at dy -1.5, motor
pads at (-0.2, +3.5).

Anchors: leaf1 (93.9, 82), yaw (101.9, 82), leaf2 (109.9, 82) across the north
band; leaf3 (93.9, 120.5) untouched and leaf4 (109.9, 120.5) south. TP6/TP7
moved clear of the new motor pads.

DRC: no clearance and no courtyard violations; 275 unconnected (nothing routed
yet) and 296 warnings that are the known lib_footprint_mismatch set plus 6 silk
edge-clearance. The 20 min-hole errors are gone - user set min through hole to
0.2 mm.

MIGRATION.md records the pattern table, the two consequences of the uniform
orientation (north channels' motor pads face the aperture; encoder FFCs no
longer sit by their channel), the parts still parked off-board, and the ordered
silkscreen plan (library text fix -> Update Footprints from Library -> Repeat
Layout), since Konnect has no tool for footprint text.

Co-Authored-By: Claude Opus 5 (1M context) <noreply@anthropic.com>
Parts:
- removed C28: 100nF, MC3_COL_MAIN:C_0402_1005Metric, symbol Device:C
- removed C29: 4.7uF, MC3_COL_MAIN:C_0603_1608Metric, symbol Device:C
- removed C30: 4.7nF, MC3_COL_MAIN:C_0402_1005Metric, symbol Device:C
- removed D4: PESD1CAN, MC3_COL_MAIN:SOT-23, symbol Device:D_TVS_Dual_AAC
- removed FB3: 600R@100MHz, MC3_COL_MAIN:L_0603_1608Metric, symbol Device:FerriteBead
- removed J12: CAN, MC3_COL_MAIN:SolderPads_3x_2.2x1.4mm_P2.6mm, symbol Connector_Generic:Conn_01x03
- removed JP1: TERM, MC3_COL_MAIN:SolderJumper-2_P1.3mm_Bridged_RoundedPad1.0x1.5mm, symbol Jumper:SolderJumper_2_Bridged
- removed R31, R32: 62R, MC3_COL_MAIN:R_0402_1005Metric, symbol Device:R
- removed U8: TJA1051T/3, MC3_COL_MAIN:SOIC-8_3.9x4.9mm_P1.27mm, symbol Interface_CAN_LIN:TJA1051T-3
- added C17: 4.7uF, MC3_COL_MAIN:C_0603_1608Metric, symbol Device:C
- added FB2: 600R@100MHz, MC3_COL_MAIN:L_0603_1608Metric, symbol Device:FerriteBead
- added J3: ENC_leaf1, MC3_COL_MAIN:Panasonic_AYF530435_FFC-4P_P0.5mm, symbol Connector_Generic:Conn_01x04
- added J4: ENC_leaf2, MC3_COL_MAIN:Panasonic_AYF530435_FFC-4P_P0.5mm, symbol Connector_Generic:Conn_01x04
- added J5: ENC_leaf3, MC3_COL_MAIN:Panasonic_AYF530435_FFC-4P_P0.5mm, symbol Connector_Generic:Conn_01x04
- added J6: ENC_leaf4, MC3_COL_MAIN:Panasonic_AYF530435_FFC-4P_P0.5mm, symbol Connector_Generic:Conn_01x04
- added R12, R13, R14, R15: 10k, MC3_COL_MAIN:R_0402_1005Metric, symbol Device:R
Connections:
- net +3V3: now also R12.1, R13.1, R14.1, R15.1
- net GND: now also C17.2, J3.2 (Pin_2), J4.2 (Pin_2), J5.2 (Pin_2), J6.2 (Pin_2)
- net VM: now also FB2.1
- new net ENC_leaf1: J3.3 (Pin_3), R12.2
- new net ENC_leaf2: J4.3 (Pin_3), R13.2
- new net ENC_leaf3: J5.3 (Pin_3), R14.2
- new net ENC_leaf4: J6.3 (Pin_3), R15.2
- new net VSENS: C17.1, FB2.2, J3.1 (Pin_1), J4.1 (Pin_1), J5.1 (Pin_1), J6.1 (Pin_1)
- no-connect marks 0 -> 4
Other:
- note added: "Encoder interface - four 0.5 mm FFCs, one per leaf, to the LX34311 sensor boards (COL-COTS-0016). Contract: VIN 4-6 V from VM, GND, SIG open-drain pulled to +3V3 here (10k), spare unassigned. Vault: Main-Board-01 Encoder Interface / Connectors. Motor pads are on the MotorChannel sheet; supply pads on Power."
- note added: "Review 2026-08-22: FFC VIN now from VSENS = VM filtered by FB61 + C63."
- note removed: "CAN - machine control link (decision 2026-08-22; vault Control Electronics open item). STM32F412 CAN1 (PA11 RX / PA12 TX) -> TJA1051T/3 -> split termination (2x62R + 4.7nF, solder-jumper JP70 bridged) + PESD1CAN -> pads CANH/CANL/GND. Classic CAN 500 kbit/s. Layout: CANH/CANL as a tight pair, transceiver and termination next to the pads, D70 nearest the pads."
