File: boards/MC3_COL_MAIN_V1.0/_restore_backup_2026-08-22T14-11-53-608/MC3_COL_MAIN_V1.0.kicad_pcb (KiCad board)
At the start: 4 copper layers, 66 x 66 mm, 101 parts, among them J1 SUPPLY_IN, J10 MOTOR, J11 MOTOR, J12 CAN, J2 SWD, J3 ENC_leaf1, J4 ENC_leaf2, J5 ENC_leaf3, J6 ENC_leaf4, J7 MOTOR, J8 MOTOR, J9 MOTOR, Q1 AO4407C, SW1 SKRKAEE020, U1 AMS1117-3.3, U2 STM32F412RET6, U3 DRV8214RTER, U4 DRV8214RTER, U5 DRV8214RTER, U6 DRV8214RTER, U7 DRV8214RTER, U8 TJA1051T/3, Y1 8MHz

Commit message: PCB placement pass 2: all five motor channels on one uniform pattern
User decision: drop the per-channel rotation. leaf3 (arranged by hand in the
GUI) is the pattern; leaf1, leaf2, leaf4 and yaw are now byte-identical copies
of its relative geometry at the same orientation - driver at -90, top row of
0402s at dy -3.5, 1 uF VM cap at (-3, +1), address straps at dy -1.5, motor
pads at (-0.2, +3.5).

Anchors: leaf1 (93.9, 82), yaw (101.9, 82), leaf2 (109.9, 82) across the north
band; leaf3 (93.9, 120.5) untouched and leaf4 (109.9, 120.5) south. TP6/TP7
moved clear of the new motor pads.

DRC: no clearance and no courtyard violations; 275 unconnected (nothing routed
yet) and 296 warnings that are the known lib_footprint_mismatch set plus 6 silk
edge-clearance. The 20 min-hole errors are gone - user set min through hole to
0.2 mm.

MIGRATION.md records the pattern table, the two consequences of the uniform
orientation (north channels' motor pads face the aperture; encoder FFCs no
longer sit by their channel), the parts still parked off-board, and the ordered
silkscreen plan (library text fix -> Update Footprints from Library -> Repeat
Layout), since Konnect has no tool for footprint text.

Co-Authored-By: Claude Opus 5 (1M context) <noreply@anthropic.com>
Parts:
- moved R29 45.6 mm to (113.2, 122.0), turned to 0 degrees
- moved R30 43.5 mm to (112.0, 120.5), turned to 0 degrees
- moved C27 41.7 mm to (113.6, 118.6), turned to 0 degrees
- moved C26 41.1 mm to (115.6, 120.6), turned to 0 degrees
- moved J11 39.3 mm to (120.2, 120.2)
- moved R28 39.0 mm to (112.0, 116.5)
- moved U7 36.0 mm to (108.1, 117.5), turned to 45 degrees
- moved R25 30.9 mm to (80.7, 113.5)
- moved C25 28.1 mm to (82.1, 114.2)
- moved R27 27.1 mm to (82.1, 112.1), turned to 0 degrees
- moved R26 26.7 mm to (80.7, 115.5)
- moved J10 25.9 mm to (84.0, 120.5)
- moved U6 25.1 mm to (85.5, 114.5), turned to 0 degrees
- moved C1 23.0 mm to (113.9, 101.0)
- moved C2 23.0 mm to (119.5, 107.5)
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