File: boards/MC3_COL_MAIN_V1.1/MotorChannel.kicad_sch (KiCad schematic)
At the start: 8 parts, among them J7 MOTOR, U3 DRV8214RTER

Commit message: V1.1: J13 machine-harness FFC (TE 84952-6, 1.0 mm 6-way) - YAW_OUT1/2 via new OUT1/OUT2 sheet pins, VIN_PAD/GND/CANH/CANL; ERC 0 errors
Changed lines of the file:
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@@
 	(generator_version "10.0")
 	(paper "A4")
-	(text "Motor channel - one per leaf, instantiated x4. Implements: COL-COTS-0028 (DRV8214, integrated current sense + ripple counting) - vault Main-Board-01 Motor Channel. Layout: docs/design/parts/DRV8214.md. PAD + GND to the GND plane via thermal vias. VREF = +3V3 (TI typical app). PROVISIONAL: R_IPROPI, pull-ups."
-		(exclude_from_sim no)
-		(at 40 30 0)
-		(effects
-			(font
-				(size 1.5 1.5)
-			)
-		)
-	)
-	(text "Review 2026-08-22: R_IPROPI 6.8k -> hardware current trip 1.99 A (was 8.45k -> 1.60 A)."
-		(exclude_from_sim no)
-		(at 94.742 120.316 0)
-		(effects
-			(font
-				(size 1.5 1.5)
-			)
-		)
-	)
-	(text "A1/A0 tri-level address straps are set per instance on the root sheet (GND / +3V3)."
-		(exclude_from_sim no)
-		(at 94.742 115.316 0)
-		(effects
-			(font
-				(size 1.5 1.5)
-			)
-		)
-	)
 	(wire
 		(pts
-			(xy 87.63 82.55) (xy 85.09 82.55)
+			(xy 87.63 82.55)
+			(xy 85.09 82.55)
 		)
 		(stroke
@@
 	(wire
 		(pts
-			(xy 97.79 64.77) (xy 97.79 63.5)
+			(xy 97.79 64.77)
+			(xy 97.79 63.5)
 		)
 		(stroke
@@
 	(wire
 		(pts
-			(xy 87.63 80.01) (xy 85.09 80.01)
+			(xy 87.63 80.01)
+			(xy 85.09 80.01)
 		)
 		(stroke
@@
 	(wire
 		(pts
-			(xy 144.78 69.85) (xy 144.78 68.58)
+			(xy 144.78 69.85)
+			(xy 144.78 68.58)
 		)
 		(stroke
@@
 	(wire
 		(pts
-			(xy 134.62 69.85) (xy 134.62 68.58)
+			(xy 134.62 69.85)
+			(xy 134.62 68.58)
 		)
 		(stroke
@@
 	(wire
 		(pts
-			(xy 87.63 77.47) (xy 85.09 77.47)
+			(xy 87.63 77.47)
+			(xy 85.09 77.47)
 		)
 		(stroke
@@
 	(wire
 		(pts
-			(xy 124.46 96.52) (xy 124.46 95.25)
+			(xy 124.46 96.52)
+			(xy 124.46 95.25)
 		)
 		(stroke
@@
 		)
 	)
+	(text "Motor channel - one per leaf, instantiated x4. Implements: COL-COTS-0028 (DRV8214, integrated current sense + ripple counting) - vault Main-Board-01 Motor Channel. Layout: docs/design/parts/DRV8214.md. PAD + GND to the GND plane via thermal vias. VREF = +3V3 (TI typical app). PROVISIONAL: R_IPROPI, pull-ups."
+		(at 40 30 0)
+		(effects
+			(font
+				(size 1.5 1.5)
+			)
+		)
+	)
+	(text "Review 2026-08-22: R_IPROPI 6.8k -> hardware current trip 1.99 A (was 8.45k -> 1.60 A)."
+		(at 94.742 120.316 0)
+		(effects
+			(font
+				(size 1.5 1.5)
+			)
+		)
+	)
+	(text "A1/A0 tri-level address straps are set per instance on the root sheet (GND / +3V3)."
+		(at 94.742 115.316 0)
+		(effects
+			(font
+				(size 1.5 1.5)
+			)
+		)
+	)
 	(label "+3V3"
 		(at 119.38 54.61 0)
@@
 		(shape input)
 		(at 87.63 72.39 180)
+		(effects
+			(font
+				(size 1.27 1.27)
+			)
+			(justify right)
+		)
+	)
+	(hierarchical_label "OUT1"
+		(shape output)
+		(at 144.78 95.25 180)
+		(effects
+			(font
+				(size 1.27 1.27)
+			)
+			(justify right)
+		)
+	)
+	(hierarchical_label "OUT2"
+		(shape output)
+		(at 144.78 97.79 180)
 		(effects
 			(font
@@
 		(at 134.62 64.77 0)
 		(unit 1)
-		(body_style 1)
 		(exclude_from_sim no)
 		(in_bom yes)
 		(on_board yes)
-		(in_pos_files yes)
 		(dnp no)
 		(property "Reference" "R17"
@@
 			)
 		)
+		(body_style 1)
+		(in_pos_files yes)
 		(pin "1"
 		)
@@
 		(at 144.78 64.77 0)
 		(unit 1)
-		(body_style 1)
 		(exclude_from_sim no)
 		(in_bom yes)
 		(on_board yes)
-		(in_pos_files yes)
 		(dnp no)
 		(property "Reference" "R18"
@@
 			)
 		)
+		(body_style 1)
+		(in_pos_files yes)
 		(pin "1"
 		)
@@
 		(at 124.46 91.44 0)
 		(unit 1)
-		(body_style 1)
 		(exclude_from_sim no)
 		(in_bom yes)
 		(on_board yes)
-		(in_pos_files yes)
 		(dnp no)
 		(property "Reference" "R16"
@@
 			)
 		)
+		(body_style 1)
+		(in_pos_files yes)
 		(pin "2"
 		)
@@
 		(at 97.79 95.25 0)
 		(unit 1)
-		(body_style 1)
 		(exclude_from_sim no)
 		(in_bom yes)
 		(on_board yes)
-		(in_pos_files yes)
 		(dnp no)
 		(property "Reference" "#PWR011"
@@
 			)
 		)
+		(body_style 1)
+		(in_pos_files yes)
 		(pin "1"
 		)
@@
 		(at 74.93 58.42 0)
 		(unit 1)
-		(body_style 1)
 		(exclude_from_sim no)
 		(in_bom yes)
 		(on_board yes)
-		(in_pos_files yes)
 		(dnp no)
 		(property "Reference" "C18"
@@
 			)
 		)
+		(body_style 1)
+		(in_pos_files yes)
 		(pin "2"
 		)
@@
 		(at 90.17 58.42 0)
 		(unit 1)
-		(body_style 1)
 		(exclude_from_sim no)
 		(in_bom yes)
 		(on_board yes)
-		(in_pos_files yes)
 		(dnp no)
 		(property "Reference" "C31"
@@
 			)
 		)
+		(body_style 1)
+		(in_pos_files yes)
 		(pin "1"
 		)
@@
 		(at 100.33 80.01 0)
 		(unit 1)
-		(body_style 1)
 		(exclude_from_sim no)
 		(in_bom yes)
 		(on_board yes)
-		(in_pos_files yes)
 		(dnp no)
 		(property "Reference" "U3"
@@
 			)
 		)
+		(body_style 1)
+		(in_pos_files yes)
 		(pin "13"
 		)
@@
 		(at 149.86 95.25 0)
 		(unit 1)
-		(body_style 1)
 		(exclude_from_sim no)
 		(in_bom yes)
 		(on_board yes)
-		(in_pos_files yes)
 		(dnp no)
 		(property "Reference" "J7"
@@
 			)
 		)
+		(body_style 1)
+		(in_pos_files yes)
 		(pin "2"
 		)
@@
 		(at 102.87 64.77 0)
 		(unit 1)
-		(body_style 1)
 		(exclude_from_sim no)
 		(in_bom yes)
 		(on_board yes)
-		(in_pos_files yes)
 		(dnp no)
 		(property "Reference" "#PWR012"
@@
 			)
 		)
+		(body_style 1)
+		(in_pos_files yes)
 		(pin "1"
 		)
@@
 		(at 119.38 58.42 0)
 		(unit 1)
-		(body_style 1)
 		(exclude_from_sim no)
 		(in_bom yes)
 		(on_board yes)
-		(in_pos_files yes)
 		(dnp no)
 		(property "Reference" "C19"
@@
 			)
 		)
+		(body_style 1)
+		(in_pos_files yes)
 		(pin "1"
 		)
