File: boards/MC3_COL_MAIN_V1.1/MC3_COL_MAIN_V1.1.kicad_pcb (KiCad board)
At the start: 4 copper layers, 66 x 66 mm, 157 parts, among them J1 SUPPLY_IN, J10 MOTOR, J11 MOTOR, J12 CAN, J13 HARNESS_FFC_6P, J2 SWD, J3 ENC_leaf1, J4 ENC_leaf2, J5 ENC_leaf3, J6 ENC_leaf4, J7 MOTOR, J8 MOTOR, J9 MOTOR, Q1 AO4421, SW1 SKRKAEE020, U1 AMS1117-3.3, U10 GP1S094HCZ0F, U11 GP1S094HCZ0F, U12 LM61460AANRJRR, U2 STM32U595RJT6, U3 DRV8214RTER, U4 DRV8214RTER, U5 DRV8214RTER, U6 DRV8214RTER, U7 DRV8214RTER, U8 TJA1051T/3, U9 AEDR-8300-1Q0, Y1 8MHz

Commit message: V1.1: bottom GND pour restored (deleted in a board session; same outline/settings as the fork)
Connections:
- R12 pad 2: ENC_leaf1 -> ENC_leaf2
- R13 pad 2: ENC_leaf2 -> ENC_leaf1
- R14 pad 2: ENC_leaf3 -> ENC_leaf4
- R15 pad 2: ENC_leaf4 -> ENC_leaf3
- U2 pad 14: ENC_leaf3 -> ENC_leaf4
- U2 pad 15: ENC_leaf4 -> ENC_leaf3
- U2 pad 17: ENC_leaf1 -> ENC_leaf2
- U2 pad 29: ENC_leaf2 -> ENC_leaf1
Routing:
- net ENC_leaf3: track 22.0 -> 53.6 mm, vias 3 -> 2
- net ENC_leaf4: track 53.2 -> 22.2 mm, vias 2 -> 3
- net ENC_leaf2: track 49.9 -> 80.2 mm
- net ENC_leaf1: track 80.2 -> 49.9 mm
- net RC_OUT_leaf4: track 26.0 -> 38.4 mm, vias 2 -> 3
- net PH_leaf3: track 37.9 -> 36.6 mm
- net /MCU/YAW_HOME: track 63.4 -> 64.2 mm
- added copper zone on B.Cu, net GND
