File: boards/MC3_COL_MAIN_V1.1/Power.kicad_sch (KiCad schematic)
At the start: 34 parts, among them J1 SUPPLY_IN, Q1 AO4421, U1 AMS1117-3.3, U12 LM61460AANRJRR

Commit message: Vault consolidation: Main-Board-02 rung folded back into Main-Board-01
Nothing was built at V1.0, so the 24 V revision never justified a rung bump.
Main-Board-01 now builds boards/MC3_COL_MAIN_V1.1 (24 V input); V1.0 stays in
the repo as the 5 V-only fallback revision. Repo side: CLAUDE.md rung mapping,
MIGRATION.md header and §14 pointer, LM61460 layout-note link. Vault side
(edited directly): Main-Board-01 Power rewritten as the 24 V chain, rung page
carries the V1.0→V1.1 delta/BOM/gates, Main-Board-02 folder deleted, 13 pages'
references rewritten.

Co-Authored-By: Claude Fable 5 <noreply@anthropic.com>
Parts:
- removed J1: SUPPLY_IN, MC3_COL_MAIN:SolderPads_2x_3.5x2.0mm_P4.2mm, symbol Connector_Generic:Conn_01x02
- added TP9: VIN_PAD, MC3_COL_MAIN:TestPoint_Pad_1.0x1.0mm, symbol Connector:TestPoint
Connections:
- net VIN_PAD: now also TP9.1
Changed lines of the file:
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@@
 	(text "Power - PROTOTYPE architecture (vault Main-Board-01: 5 V in -> P-FET reverse-polarity -> VM direct; 3.3 V via LDO). Incoming supply rail is an open entry gate in the vault. Net naming: vault VIN_RAW == KiCad VM (same copper). Sensor VIN (encoder FFCs) also runs from VM (LX34311 needs 4-6 V)."
 		(exclude_from_sim no)
-		(at 30 40 0)
+		(at 38.354 181.864 0)
 		(effects
 			(font
@@
 	)
 	(label "GND"
-		(at 33.02 77.47 180)
-		(effects
-			(font
-				(size 1.27 1.27)
-			)
-			(justify right bottom)
-		)
-	)
-	(label "GND"
 		(at 119.38 97.79 0)
 		(effects
@@
 	)
 	(symbol
+		(lib_id "Connector:TestPoint")
+		(at 33.02 74.93 0)
+		(unit 1)
+		(body_style 1)
+		(exclude_from_sim no)
+		(in_bom yes)
+		(on_board yes)
+		(in_pos_files yes)
+		(dnp no)
+		(property "Reference" "TP9"
+			(at 33.02 68.072 0)
+			(show_name no)
+			(do_not_autoplace no)
+			(effects
+				(font
+					(size 1.27 1.27)
+				)
+			)
+		)
+		(property "Value" "VIN_PAD"
+			(at 33.02 69.85 0)
+			(show_name no)
+			(do_not_autoplace no)
+			(effects
+				(font
+					(size 1.27 1.27)
+				)
+			)
+		)
+		(property "Footprint" "MC3_COL_MAIN:TestPoint_Pad_1.0x1.0mm"
+			(at 33.02 74.93 0)
+			(hide yes)
+			(show_name no)
+			(do_not_autoplace no)
+			(effects
+				(font
+					(size 1.27 1.27)
+				)
+			)
+		)
+		(property "Datasheet" ""
+			(at 33.02 74.93 0)
+			(hide yes)
+			(show_name no)
+			(do_not_autoplace no)
+			(effects
+				(font
+					(size 1.27 1.27)
+				)
+			)
+		)
+		(property "Description" ""
+			(at 33.02 74.93 0)
+			(show_name no)
+			(do_not_autoplace no)
+			(effects
+				(font
+					(size 1.27 1.27)
+				)
+			)
+		)
+		(pin "1"
+		)
+		(instances
+			(project "MC3_COL_MAIN_V1.1"
+				(path "/7d5f4202-d55e-4c7b-a2df-dd599db38e48/d6d9c27b-d616-4172-a586-88c2a3452975"
+					(reference "TP9")
+					(unit 1)
+				)
+			)
+		)
+	)
+	(symbol
 		(lib_id "Device:Polyfuse")
 		(at 45.72 95.25 0)
@@
 		)
 		(property "Value" "1uF"
-			(at 122.555 149.86 0)
+			(at 117.602 151.13 0)
 			(show_name no)
 			(do_not_autoplace no)
@@
 	)
 	(symbol
-		(lib_id "Connector_Generic:Conn_01x02")
-		(at 38.1 74.93 0)
-		(unit 1)
-		(body_style 1)
-		(exclude_from_sim no)
-		(in_bom yes)
-		(on_board yes)
-		(in_pos_files yes)
-		(dnp no)
-		(property "Reference" "J1"
-			(at 38.1 72.39 0)
-			(show_name no)
-			(do_not_autoplace no)
-			(effects
-				(font
-					(size 1.27 1.27)
-				)
-			)
-		)
-		(property "Value" "SUPPLY_IN"
-			(at 38.1 80.01 0)
-			(show_name no)
-			(do_not_autoplace no)
-			(effects
-				(font
-					(size 1.27 1.27)
-				)
-			)
-		)
-		(property "Footprint" "MC3_COL_MAIN:SolderPads_2x_3.5x2.0mm_P4.2mm"
-			(at 38.1 74.93 0)
-			(hide yes)
-			(show_name no)
-			(do_not_autoplace no)
-			(effects
-				(font
-					(size 1.27 1.27)
-				)
-			)
-		)
-		(property "Datasheet" ""
-			(at 38.1 74.93 0)
-			(hide yes)
-			(show_name no)
-			(do_not_autoplace no)
-			(effects
-				(font
-					(size 1.27 1.27)
-				)
-			)
-		)
-		(property "Description" ""
-			(at 38.1 74.93 0)
-			(show_name no)
-			(do_not_autoplace no)
-			(effects
-				(font
-					(size 1.27 1.27)
-				)
-			)
-		)
-		(property "Note" "Machine supply: bare pads 3.5x2.0 @4.2 mm, 20-22 AWG, whole-board current - vault Connectors, Machine Interface. Pin1 = VIN_PROT (+), Pin2 = GND. Supply rail unspecified (vault entry gate); 5 V assumed for this prototype."
-			(at 38.1 74.93 0)
-			(hide yes)
-			(show_name no)
-			(do_not_autoplace no)
-			(effects
-				(font
-					(size 1.27 1.27)
-				)
-			)
-		)
-		(pin "1"
-		)
-		(pin "2"
-		)
-		(instances
-			(project "Power"
-				(path "/62fa4f2c-604d-44f9-988f-2ce377285c9c"
-					(reference "J3")
-					(unit 1)
-				)
-			)
-			(project "MC3_COL_MAIN_V1.1"
-				(path "/7d5f4202-d55e-4c7b-a2df-dd599db38e48/d6d9c27b-d616-4172-a586-88c2a3452975"
-					(reference "J1")
-					(unit 1)
-				)
-			)
-		)
-	)
-	(symbol
 		(lib_id "Connector:TestPoint")
 		(at 195.58 110.49 0)
@@
 		)
 		(property "Value" "2.2uH XAL5030-222"
-			(at 124.714 132.842 90)
+			(at 123.952 127.508 90)
 			(show_name no)
 			(do_not_autoplace no)
