File: boards/MC3_COL_MAIN_V1.1/Power.kicad_sch (KiCad schematic)
At the start: 34 parts, among them Q1 AO4421, U1 AMS1117-3.3, U12 LM61460AANRJRR

Commit message: V1.1 schematics: per-instance Description fields on ~63 symbols
The component-docs Role source of record. Netlist unchanged, ERC 0.

Co-Authored-By: Claude Fable 5 <noreply@anthropic.com>
Other:
- note removed: "Power - PROTOTYPE architecture (vault Main-Board-01: 5 V in -> P-FET reverse-polarity -> VM direct; 3.3 V via LDO). Incoming supply rail is an open entry gate in the vault. Net naming: vault VIN_RAW == KiCad VM (same copper). Sensor VIN (encoder FFCs) also runs from VM (LX34311 needs 4-6 V)."
- note removed: "Review 2026-08-22: input path = pads (VIN_PAD) -> polyfuse F60 -> VIN_PROT (TVS D62 to GND) -> Q1 reverse-polarity FET -> VM. VM bulk C61/C62 2x22uF added (TI: sufficient bulk on VM). LDO output cap now tantalum."
- moved on the sheet: C1, C2, C3, C32, C4, C48, C49, C50, C51, C52, C53, C54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

Commit message: BOM availability audit: stale V1.0 part numbers fixed, V1.1 passives backfilled
F1 1206L200 -> 1812L075/33DR (C151170, the fuse the 24V design actually
specifies); D1 SMAJ5.0A -> SMAJ28A; Q1 AO4407C -> AO4421 (C33484) - three
turnkey landmines from the 24V conversion. D7 BZT52C12 numbered; 15 buck-era
passive lines given LCSC/MPN (copied from proven same-value lines where they
exist, formulaic Yageo/Samsung/Murata otherwise). Every fitted BOM line now
carries a part number except J2 (to be marked DNP). Netlist unchanged.

Co-Authored-By: Claude Fable 5 <noreply@anthropic.com>
Parts:
- C48, C49: MPN (none) -> GRM32ER71H106KA12L
- C50: LCSC (none) -> C1591; MPN (none) -> CL10B104KB8NNNC
- C51: LCSC (none) -> C1523
- C52, C54: LCSC (none) -> C1525; MPN (none) -> CL05B104KO5NNNC
- C53: LCSC (none) -> C15849; MPN (none) -> CL10A105KB8NNNC
- C55: MPN (none) -> 0402CG4R7C500NT
- C56, C57: LCSC (none) -> C45783; MPN (none) -> CL21A226MAQNNNE
- D1: LCSC C78401 -> (none); MPN SMAJ5.0A/TR13 -> SMAJ28A
- D7: MPN (none) -> BZT52C12
- F1: LCSC C19078716 -> C151170; MPN 1206L200/12NR -> 1812L075/33DR
- Q1: LCSC C469397 -> C33484; MPN AO4407C -> AO4421
- R41: MPN (none) -> 0402WGF1332TCE
- R42, R45: LCSC (none) -> C25741; MPN (none) -> 0402WGF1003TCE
- R43: MPN (none) -> 0402WGF8661TCE
- R44: MPN (none) -> 0402WGF0000TCE
- R46: MPN (none) -> 0402WGF2492TCE
- R47: LCSC (none) -> C11702; MPN (none) -> 0402WGF1001TCE
