File: boards/MC3_COL_MAIN_V1.1/MC3_COL_MAIN_V1.1.kicad_sch (KiCad schematic)
At the start: 9 parts

Commit message: V1.1: encoder FFC VIN on filtered VSENS, motor pads off MotorChannel, yaw nets renamed
- Connectors: encoder FFC VIN now fed from VSENS (VM through FB61 + C63);
  ENC_leaf1-4 / RC_OUT labels re-placed; SIG pull-ups to +3V3 noted on sheet
- MotorChannel: J7-J9 MOTOR pad connectors (Conn_01x02) and their OUT1/OUT2
  hierarchical labels removed from the shared sheet
- MCU: ENC_leaf1-4 global labels re-placed; sheet notes carried over
- Root: H5 SLOT-PASSTHRU mounting hole removed
- PCB: yaw motor nets YAW_OUT* -> /yaw/OUT*; CANH/CANL pad assignment swapped;
  VSENS/VM net reassignments and follow-up routing (~106 segments, 12 vias,
  zone edits) to match the schematic

Co-Authored-By: Claude Fable 5 <noreply@anthropic.com>
Parts:
- removed H5: SLOT-PASSTHRU, MC3_COL_MAIN:SlotNPTH_PassThrough, symbol Mechanical:MountingHole
Changed lines of the file:
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@@
-	(symbol
-		(lib_id "Mechanical:MountingHole")
-		(at 93.98 110.49 0)
-		(unit 1)
-		(body_style 1)
-		(exclude_from_sim no)
-		(in_bom yes)
-		(on_board yes)
-		(in_pos_files yes)
-		(dnp no)
-		(property "Reference" "H5"
-			(at 93.98 105.41 0)
-			(show_name no)
-			(do_not_autoplace no)
-			(effects
-				(font
-					(size 1.27 1.27)
-				)
-			)
-		)
-		(property "Value" "SLOT-PASSTHRU"
-			(at 93.98 107.315 0)
-			(show_name no)
-			(do_not_autoplace no)
-			(effects
-				(font
-					(size 1.27 1.27)
-				)
-			)
-		)
-		(property "Footprint" "MC3_COL_MAIN:SlotNPTH_PassThrough"
-			(at 93.98 110.49 0)
-			(hide yes)
-			(show_name no)
-			(do_not_autoplace no)
-			(effects
-				(font
-					(size 1.27 1.27)
-				)
-			)
-		)
-		(property "Datasheet" ""
-			(at 93.98 110.49 0)
-			(hide yes)
-			(show_name no)
-			(do_not_autoplace no)
-			(effects
-				(font
-					(size 1.27 1.27)
-				)
-			)
-		)
-		(property "Description" ""
-			(at 93.98 110.49 0)
-			(show_name no)
-			(do_not_autoplace no)
-			(effects
-				(font
-					(size 1.27 1.27)
-				)
-			)
-		)
-		(property "Note" "PROVISIONAL - wire pass-through slot for temporarily routing the yaw motor leads to the power/CAN pad area on the back. Placeholder circular 2.5mm NPTH: in the footprint editor set Hole shape = Oval and tune size; position in layout. Delete when the yaw lead routing is permanent"
-			(at 93.98 110.49 0)
-			(hide yes)
-			(show_name no)
-			(do_not_autoplace no)
-			(effects
-				(font
-					(size 1.27 1.27)
-				)
-			)
-		)
-		(instances
-			(project "MC3_COL_MAIN_V1.1"
-				(path "/7d5f4202-d55e-4c7b-a2df-dd599db38e48"
-					(reference "H5")
-					(unit 1)
-				)
-			)
-		)
-	)
 	(symbol
 		(lib_id "Mechanical:MountingHole")

Commit message: V1.1: power routing pass — 24V chain + buck routed, stale-net/short fixes, VQFN corner pads fused, yaw OUT hier labels restored
- Board: VIN chain and buck cell routed (VIN_SW vias at Q1 source, SW between
  pads 8/9, boot via In2); ENC_leaf1 via at (83.9,97.075) renamed to ENC_leaf2;
  stray GND via under U1 strap deleted; VSENS via moved off the R32 rim arc;
  YAW_ENC_B gap closed at U9.1.
- MotorChannel.kicad_sch: OUT1/OUT2 hierarchical labels (passive) restored on
  the driver output wires; netlist verified YAW_OUT1/2 = U7 OUT + J13 5/6.
- VQFN-HR14_RJR_TEX: UL corner L-extensions were net-less F.Cu polygons over
  pads 1/5/9/11 (DRC overlap noise, parser-breaking width-0 strokes); fused
  into single rect pads covering the exact union; polys deleted. Board still
  carries the old embedded copy - Update Footprint on U12 pending.

Co-Authored-By: Claude Fable 5 <noreply@anthropic.com>
Changed lines of the file:
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@@
 			)
 		)
-		(pin "OUT1" passive
+		(pin "OUT1" input
 			(at 102.87 90.17 0)
 			(effects
@@
 			)
 		)
-		(pin "OUT2" passive
+		(pin "OUT2" input
 			(at 102.87 92.71 0)
 			(effects
@@
 			)
 		)
-		(pin "OUT1" passive
+		(pin "OUT1" input
 			(at 257.81 88.9 0)
 			(effects
@@
 			)
 		)
-		(pin "OUT2" passive
+		(pin "OUT2" input
 			(at 257.81 91.44 0)
 			(effects
@@
 			)
 		)
-		(pin "OUT1" passive
+		(pin "OUT1" input
 			(at 204.47 87.63 0)
 			(effects
@@
 			)
 		)
-		(pin "OUT2" passive
+		(pin "OUT2" input
 			(at 204.47 90.17 0)
 			(effects
@@
 			)
 		)
-		(pin "OUT1" passive
+		(pin "OUT1" input
 			(at 52.07 90.17 0)
 			(effects
@@
 			)
 		)
-		(pin "OUT2" passive
+		(pin "OUT2" input
 			(at 52.07 92.71 0)
 			(effects
@@
 			)
 		)
-		(pin "OUT1" passive
+		(pin "OUT1" input
 			(at 153.67 88.9 0)
 			(effects
@@
 			)
 		)
-		(pin "OUT2" passive
+		(pin "OUT2" input
 			(at 153.67 91.44 0)
 			(effects

Commit message: V1.1 schematics: per-instance Description fields on ~63 symbols
The component-docs Role source of record. Netlist unchanged, ERC 0.

Co-Authored-By: Claude Fable 5 <noreply@anthropic.com>
Other:
- note removed: "Address straps per SLVSH04 Table 8-28: leaf1 0/0 -> 0x60, leaf2 0/1 -> 0x64, leaf3 1/0 -> 0x6C, leaf4 1/1 -> 0x70, yaw Z/0 -> 0x66 (write addresses). High straps via 2.2k per TI; low straps tied to GND; Hi-Z left open."
- note removed: "MC3_COL_MAIN_V1.0 - MC3 collimator main control board. Vault build rung: Projects/MC3 Collimator/05 Builds/Main-Board-01. Four leaf channels fitted (DRV8214, COL-COTS-0028); yaw reserved at the MCU only. A1/A0 I2C address straps per leaf: leaf1 GND/GND, leaf2 GND/+3V3, leaf3 +3V3/GND, leaf4 +3V3/+3V3 (PROVISIONAL). Net naming: vault V3_3 == +3V3, vault VIN_RAW == VM."
- note removed: "yaw channel fitted 2026-08-22 (user decision; vault still says reserved-only - update owed). Same DRV8214 block; assumed inside the part's limits until the yaw motor is selected. Address A1 = Hi-Z (open), A0 = GND."
Changed lines of the file:
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@@
 	(generator_version "10.0")
 	(paper "A4")
-	(text "yaw channel fitted 2026-08-22 (user decision; vault still says reserved-only - update owed). Same DRV8214 block; assumed inside the part's limits until the yaw motor is selected. Address A1 = Hi-Z (open), A0 = GND."
-		(exclude_from_sim no)
-		(at 20 195 0)
-		(effects
-			(font
-				(size 1.5 1.5)
-			)
-		)
-	)
-	(text "Address straps per SLVSH04 Table 8-28: leaf1 0/0 -> 0x60, leaf2 0/1 -> 0x64, leaf3 1/0 -> 0x6C, leaf4 1/1 -> 0x70, yaw Z/0 -> 0x66 (write addresses). High straps via 2.2k per TI; low straps tied to GND; Hi-Z left open."
-		(exclude_from_sim no)
-		(at 20 200 0)
-		(effects
-			(font
-				(size 1.5 1.5)
-			)
-		)
-	)
-	(text "MC3_COL_MAIN_V1.0 - MC3 collimator main control board. Vault build rung: Projects/MC3 Collimator/05 Builds/Main-Board-01. Four leaf channels fitted (DRV8214, COL-COTS-0028); yaw reserved at the MCU only. A1/A0 I2C address straps per leaf: leaf1 GND/GND, leaf2 GND/+3V3, leaf3 +3V3/GND, leaf4 +3V3/+3V3 (PROVISIONAL). Net naming: vault V3_3 == +3V3, vault VIN_RAW == VM."
-		(exclude_from_sim no)
-		(at 20 130 0)
-		(effects
-			(font
-				(size 1.5 1.5)
-			)
-		)
-	)
 	(no_connect
 		(at 153.67 88.9)
@@
 		(dnp no)
 		(property "Reference" "R4"
-			(at 182.88 75.438 90)
+			(at 187.452 76.708 90)
 			(show_name no)
 			(do_not_autoplace no)
@@
 			)
 		)
-		(property "Description" ""
+		(property "Description" "I²C address strap (A1/A0 tri-level) — sets this channel's DRV8214 address; map in [[Firmware-01]]."
 			(at 182.88 77.47 0)
 			(show_name no)
@@
 		(dnp no)
 		(property "Reference" "R2"
-			(at 132.08 74.168 90)
+			(at 127.254 77.47 90)
 			(show_name no)
 			(do_not_autoplace no)
@@
 			)
 		)
-		(property "Description" ""
+		(property "Description" "I²C address strap (A1/A0 tri-level) — sets this channel's DRV8214 address; map in [[Firmware-01]]."
 			(at 132.08 76.2 0)
 			(show_name no)
@@
 		(dnp no)
 		(property "Reference" "R3"
-			(at 182.88 72.898 90)
+			(at 187.452 74.168 90)
 			(show_name no)
 			(do_not_autoplace no)
@@
 			)
 		)
-		(property "Description" ""
+		(property "Description" "I²C address strap (A1/A0 tri-level) — sets this channel's DRV8214 address; map in [[Firmware-01]]."
 			(at 182.88 74.93 0)
 			(show_name no)
@@
 		(dnp no)
 		(property "Reference" "R1"
-			(at 81.28 77.978 90)
+			(at 76.708 79.248 90)
 			(show_name no)
 			(do_not_autoplace no)
@@
 			)
 		)
-		(property "Description" ""
+		(property "Description" "I²C address strap (A1/A0 tri-level) — sets this channel's DRV8214 address; map in [[Firmware-01]]."
 			(at 81.28 80.01 0)
 			(show_name no)
@@
 		(on_board yes)
 		(dnp no)
-		(fields_autoplaced yes)
 		(stroke
 			(width 0.1524)
@@
 		)
 		(property "Sheetname" "MCU"
-			(at 90 19.365 0)
+			(at 90.17 18.288 0)
 			(show_name no)
 			(do_not_autoplace no)
@@
 		(on_board yes)
 		(dnp no)
-		(fields_autoplaced yes)
 		(stroke
 			(width 0.1524)
@@
 		)
 		(property "Sheetname" "Connectors"
-			(at 160 19.365 0)
+			(at 159.766 17.78 0)
 			(show_name no)
 			(do_not_autoplace no)
@@
 		(on_board yes)
 		(dnp no)
-		(fields_autoplaced yes)
 		(stroke
 			(width 0.1524)
@@
 		)
 		(property "Sheetname" "Power"
-			(at 20 19.365 0)
-			(show_name no)
-			(do_not_autoplace no)
+			(at 19.812 18.288 0)
+			(show_name no)
+			(do_not_autoplace no)
