File: boards/MC3_COL_MAIN_V1.1/MC3_COL_MAIN_V1.1.kicad_sch (KiCad schematic)
At the start: 8 parts

Commit message: V1.1 root: restore J7-J10 motor pads lost with the yaw pad deletion
cc54c1d removed the Conn_01x02 MOTOR pad from the shared MotorChannel
sheet to drop the yaw pad. Because that sheet is instantiated five times,
the one symbol carried all five annotations (J7-J11), so deleting it took
the four leaf pads with it. The PCB kept J7-J10 (and correctly dropped
J11 - yaw now exits via J13, the machine harness FFC), leaving four
footprints on the board with no schematic symbol and eight single-node
nets in the schematic.

Restored as four root-sheet symbols wired to each leaf's OUT1/OUT2 sheet
pins, so yaw does not get one back. Same lib_id, footprint and Note field
as the originals, recovered from cc54c1d^.

Verified:
- nets 100 -> 100 (none added, none removed); nodes 479 -> 487, the eight
  new pads and nothing else
- all 8 pads match the nets already routed on the board
  (J7=/leaf1/OUT*, J8=/leaf2/*, J9=/leaf3/*, J10=/leaf4/*) - no rework
- ERC unchanged: 0 errors, same 13 warnings
- schematic/PCB parity restored: only G8 (logo) is board-only

Co-Authored-By: Claude Opus 5 (1M context) <noreply@anthropic.com>
Claude-Session: https://claude.ai/code/session_01GzLKfQYZt6tZcskNSHuqcs
Parts:
- added J10, J7, J8, J9: MOTOR, MC3_COL_MAIN:SolderPads_2x_2.2x1.4mm_P2.6mm, symbol Connector_Generic:Conn_01x02
Connections:
- net leaf1/OUT1: now also J7.1 (Pin_1)
- net leaf1/OUT2: now also J7.2 (Pin_2)
- net leaf2/OUT1: now also J8.1 (Pin_1)
- net leaf2/OUT2: now also J8.2 (Pin_2)
- net leaf3/OUT1: now also J9.1 (Pin_1)
- net leaf3/OUT2: now also J9.2 (Pin_2)
- net leaf4/OUT1: now also J10.1 (Pin_1)
- net leaf4/OUT2: now also J10.2 (Pin_2)
